File: z80_schematic.kicad_sch (KiCad schematic)
At the start: 28 parts, among them SW1 SW_Push, SW2 SW_Push, U1 Z80CPU, U2 Z84C20, U3 TC551001CP-70L, U4 AT28C64B-15PU, U6 NE555P, U7 SN74AC00N

Commit message: 2
Parts:
- removed R11: 1k, symbol Device:R
- added C1, C12, C13: 100n, symbol Device:C
- added R1: 1k, symbol Device:R
- added U10: SN74ACT08N, Package_DIP:DIP-14_W7.62mm_Socket_LongPads, symbol Custom_symbole:SN74ACT08N
- added U8: SN74AC32, Package_DIP:DIP-14_W7.62mm_Socket_LongPads, symbol Custom_symbole:SN74AC32
- added U9: 74HCT273, Package_DIP:DIP-20_W7.62mm_Socket_LongPads, symbol 74xx:74HCT273
- U1: footprint (none) -> Package_DIP:DIP-40_W15.24mm_Socket_LongPads
- U2: footprint Package_DIP:DIP-40_W15.24mm -> Package_DIP:DIP-40_W15.24mm_Socket_LongPads
- U3: footprint Package_DIP:DIP-32_W15.24mm -> Package_DIP:DIP-32_W15.24mm_Socket_LongPads
- U4: footprint 28P6_ATM -> Package_DIP:DIP-28_W15.24mm_Socket_LongPads
- U5: value ~ -> HEF4555B; footprint Package_DIP:DIP-16_W7.62mm_LongPads -> Package_DIP:DIP-16_W7.62mm_Socket_LongPads
- U6: footprint Package_DIP:DIP-8_W7.62mm -> Package_DIP:DIP-8_W7.62mm_Socket_LongPads
- U7: footprint N14 -> Package_DIP:DIP-14_W7.62mm_Socket_LongPads
Connections:
- net +5V: now also C1.2, C12.2, C13.2, R1.2, U10.14 (VDD), U8.14 (VDD), U9.20 (VCC); no longer U3.30 (CE2)
- net ADR0: now also U9.3 (D0)
- net ADR1: now also U9.4 (D1)
- net ADR12: now also U5.14 (A_{0B})
- net ADR13: now also U5.13 (A_{1B})
- net DATA0: now also U10.1 (1A)
- net GND: now also C1.1, C12.1, C13.1, U10.7 (GND), U8.7 (GND), U9.10 (GND); no longer U5.13 (A_{1B}), U5.14 (A_{0B})
- net ~{I/O_CE}: now also U7.6 (2Y); no longer U7.8 (3Y)
- net ~{RAM_CE}: now also U3.22 (~{CE1}), U7.8 (3Y); no longer U7.6 (2Y)
- net ~{RESET_SIGNAL}: now reaches C3.1, R3.1, SW1.2, U1.26 (~{RESET})
- net ~{RESET_SIGNAL}: now also U9.1 (~{Mr})
- net RAM_PAGE_SEL: now reaches U5.11 (Out_1B)
- net RAM_PAGE_SEL: now also U10.2 (1B)
- net I/O_SUB_SEL: now reaches U5.12 (Out_0B)
- net I/O_SUB_SEL: now also U7.5 (2B)
- net I/O_SEL: now reaches U5.15 (~{EN_B})
- net I/O_SEL: now also U5.5 (Out_1A), U7.4 (2A)
- net ADR14: now reaches U1.4 (A14), U5.2 (A_{0A})
- net ADR14: now also U3.3 (A14)
- net ADR15: now reaches U1.5 (A15), U5.3 (A_{1A})
- net EEPROM_SEL: now reaches U5.4 (Out_0A), U7.1 (1A), U7.2 (1B)
- net RAM_SEL: now reaches U7.10 (3B), U7.9 (3A)
- net RAM_SEL: now also U8.3 (1Y); no longer U5.6 (Out_2A)
- net RAM_PAGE_SEL_1: now reaches U3.2 (A16)
- net RAM_PAGE_SEL_1: now also U9.5 (Q1)
- net RAM_PAGE_SEL_0: now reaches U3.31 (A15)
- net RAM_PAGE_SEL_0: now also U9.2 (Q0)
- net ~{SW_RAM_CE}: no longer names the net of U7.11 (4Y)
- net ~{SW_RAM_CE}: no longer U3.22 (~{CE1})
- new net: R1.1, U3.30 (CE2)
- new net RAM_PAGE_CLK: U10.3 (1Y), U9.11 (Cp)
- new net RAM_SEL_1: U5.6 (Out_2A), U8.1 (1A)
- new net RAM_SEL_2: U5.7 (Out_3A), U8.2 (1B)
- now unconnected: U7.12 (4A), U7.13 (4B)
Other:
- note added: "ADDRESS DECODE"
- note added: "ADDRESS SPACE (64kB, podzielone na 16kB segmenty) 0000 - 3FFF EEPROM (tylko dolna połowa adresów, 8kB, trzeba dodać większy chip) 4000 - 7FFFF I/O + paging RAMu (Adresy dalej podzielone na 4 multiplekserem (4kB)) I/O chip: 4000 Port A, Data 4001 Port B, Data 4002 Port A, Command 4003 Port B, Command RAM paging (D flip-flop) strona ustawiana adresem, zegar wywołany linią danych (DATA 0) po wybrani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"
- note added: "ADDRESS SPACE SIGNAL"
- note added: "CPU BLOCK"
- note removed: "ADDRESS SPACE 0 - 16383 EEPROM (tylko dolna połowa adresów, 8kB) 16384 - 32767 DEFAULT RAM (tylko dolna połowa adresów, 8kB) 32768 - 49151 I/O i inne 49152 - 65535 SWITCH RAM"
- title: (none) -> Komputer Z80
- moved on the sheet: C10, C11, C2, C3, C4, C5, C6, C7, C8, C9, R10, R2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

Commit message: ROM divide
Parts:
- added C14: 100n, symbol Device:C
- added U11: AT28C64B-15PU, Package_DIP:DIP-28_W15.24mm_Socket_LongPads, symbol Custom_symbole:AT28C64B-15PU
Connections:
- net +5V: now also C14.1, U11.27 (~{WE}), U11.28 (VCC)
- net ADR0: now also U11.10 (A0)
- net ADR1: now also U11.9 (A1)
- net ADR10: now also U11.21 (A10)
- net ADR11: now also U11.23 (A11)
- net ADR12: now also U11.2 (A12)
- net ADR13: now also U7.1 (1A), U8.5 (2B)
- net ADR2: now also U11.8 (A2)
- net ADR3: now also U11.7 (A3)
- net ADR4: now also U11.6 (A4)
- net ADR5: now also U11.5 (A5)
- net ADR6: now also U11.4 (A6)
- net ADR7: now also U11.3 (A7)
- net ADR8: now also U11.25 (A8)
- net ADR9: now also U11.24 (A9)
- net DATA0: now also U11.11 (I/O0)
- net DATA1: now also U11.12 (I/O1)
- net DATA2: now also U11.13 (I/O2)
- net DATA3: now also U11.15 (I/O3)
- net DATA4: now also U11.16 (I/O4)
- net DATA5: now also U11.17 (I/O5)
- net DATA6: now also U11.18 (I/O6)
- net DATA7: now also U11.19 (I/O7)
- net EEPROM_SEL: now also U7.12 (4A), U7.13 (4B); no longer U7.1 (1A)
- net GND: now also C14.2, U11.14 (GND)
- net ~{READ}: now also U11.22 (~{OE})
- net EEPROM_BIOS_SUB_SEL: now reaches U7.11 (4Y)
- net EEPROM_BIOS_SUB_SEL: now also U8.4 (2A)
- net ~{EEPROM_CE_BIOS}: now reaches U8.6 (2Y)
- net ~{EEPROM_CE_BIOS}: now also U4.20 (~{CE})
- net ~{EEPROM_CE} renamed ~{EEPROM_CE_PROGRAM}
- net ~{EEPROM_CE_PROGRAM}: now also U11.20 (~{CE}); no longer U4.20 (~{CE})
Other:
- note added: "ADDRESS SPACE (64kB, podzielone na 16kB segmenty) 0000 - 3FFF EEPROM 0000 - 1FFF EEPROM BIOS 2000 - 3FFF EEPROM wymienny 4000 - 7FFFF I/O + paging RAMu (Adresy dalej podzielone na 4 multiplekserem (4kB)) I/O chip: 4000 Port A, Data 4001 Port B, Data 4002 Port A, Command 4003 Port B, Command RAM paging (D flip-flop) strona ustawiana adresem, zegar wywołany linią danych (DATA 0) po wybraniu adresów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"
- note removed: "ADDRESS SPACE (64kB, podzielone na 16kB segmenty) 0000 - 3FFF EEPROM (tylko dolna połowa adresów, 8kB, trzeba dodać większy chip) 4000 - 7FFFF I/O + paging RAMu (Adresy dalej podzielone na 4 multiplekserem (4kB)) I/O chip: 4000 Port A, Data 4001 Port B, Data 4002 Port A, Command 4003 Port B, Command RAM paging (D flip-flop) strona ustawiana adresem, zegar wywołany linią danych (DATA 0) po wybrani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"
- moved on the sheet: C8, R1, U3

Commit message: Version 2.0
Parts:
- removed U10: SN74ACT08N, Package_DIP:DIP-14_W7.62mm_Socket_LongPads, symbol Custom_symbole:SN74ACT08N
- removed U11, U4: AT28C64B-15PU, Package_DIP:DIP-28_W15.24mm_Socket_LongPads, symbol Custom_symbole:AT28C64B-15PU
- removed U5: HEF4555B, Package_DIP:DIP-16_W7.62mm_Socket_LongPads, symbol Custom_symbole:HEF4555B
- removed U7: SN74AC00N, Package_DIP:DIP-14_W7.62mm_Socket_LongPads, symbol Custom_symbole:SN74AC00N
- removed U8: SN74AC32, Package_DIP:DIP-14_W7.62mm_Socket_LongPads, symbol Custom_symbole:SN74AC32
- removed U9: 74HCT273, Package_DIP:DIP-20_W7.62mm_Socket_LongPads, symbol 74xx:74HCT273
- added C15, C16, C17, C18, C19, C20, C21: 100n, symbol Device:C
- added J1: Port_A, Connector_PinHeader_2.54mm:PinHeader_1x10_P2.54mm_Vertical, symbol Connector:Conn_01x10_Socket
- added J2: Port_B, Connector_PinHeader_2.54mm:PinHeader_1x10_P2.54mm_Vertical, symbol Connector:Conn_01x10_Socket
- added R11, R12, R13, R14, R15, R9: 1k, symbol Device:R
- added R16: 10k, symbol Device:R
- added U10: AT28C64B-15PU, 28P6_ATM, symbol Custom_symbole:AT28C64B-15PU
- added U11: W49F002, Package_DIP:DIP-32_W15.24mm_Socket_LongPads, symbol Custom_symbole:W49F002
- added U12: 74HC14, Package_SO:SO-14_3.9x8.65mm_P1.27mm, symbol 74xx:74HC14
- added U13: 74HCT273, Package_DIP:DIP-20_W7.62mm_Socket_LongPads, symbol 74xx:74HCT273
- added U14, U15, U16, U18: SN74AC32, Package_DIP:DIP-14_W7.62mm_Socket_LongPads, symbol Custom_symbole:SN74AC32
- added U17, U9: SN74ACT08N, Package_DIP:DIP-14_W7.62mm_Socket_LongPads, symbol Custom_symbole:SN74ACT08N
- added U4: EN29F040A, Package_DIP:DIP-32_W15.24mm_Socket_LongPads, symbol Custom_symbole:EN29F040A
- added U5: W27E512, Package_DIP:DIP-28_W15.24mm_Socket_LongPads, symbol Custom_symbole:W27E512
- added U7, U8: 74HC374, Package_DIP:DIP-20_W7.62mm_Socket_LongPads, symbol 74xx:74HC374
- R3: value 2k -> 10k
Connections:
- net +5V: now also C1.1, C12.1, C13.1, C15.1, C16.1, C17.1, C18.1, C19.1, C20.1, C21.1, R13.2, R14.2, R15.1, R16.1, R9.2, U10.28 (VCC), U11.32 (VCC), U12.14 (VCC), U13.20 (VCC), U14.14 (VDD), U15.14 (VDD), U16.14 (VDD), U17.14 (VDD), U18.14 (VDD), U4.32 (VCC), U5.28 (VCC), U7.20 (VCC), U8.20 (VCC), U9.14 (VDD); no longer C1.2, C12.2, C13.2
- net ADR0: now also U10.10 (A0), U11.12 (A0), U4.12 (A0), U5.10 (A0)
- net ADR1: now also U10.9 (A1), U11.11 (A1), U4.11 (A1), U5.9 (A1)
- net ADR10: now also U10.21 (A10), U11.23 (A10), U18.12 (4A), U4.23 (A10), U5.21 (A10)
- net ADR11: now also U10.23 (A11), U11.25 (A11), U18.13 (4B), U4.25 (A11), U5.23 (A11)
- net ADR12: now also U10.2 (A12), U11.4 (A12), U16.1 (1A), U4.4 (A12), U5.2 (A12)
- net ADR13: now also U16.2 (1B), U4.28 (A13), U5.26 (A13)
- net ADR14: now also U17.1 (1A), U5.27 (A14); no longer U3.3 (A14)
- net ADR15: now also U17.2 (1B), U5.1 (A15), U9.13 (4B)
- net ADR2: now also U10.8 (A2), U11.10 (A2), U14.1 (1A), U4.10 (A2), U5.8 (A2)
- net ADR3: now also U10.7 (A3), U11.9 (A3), U14.2 (1B), U4.9 (A3), U5.7 (A3)
- net ADR4: now also U10.6 (A4), U11.8 (A4), U14.4 (2A), U4.8 (A4), U5.6 (A4)
- net ADR5: now also U10.5 (A5), U11.7 (A5), U14.5 (2B), U4.7 (A5), U5.5 (A5)
- net ADR6: now also U10.4 (A6), U11.6 (A6), U14.9 (3A), U4.6 (A6), U5.4 (A6)
- net ADR7: now also U10.3 (A7), U11.5 (A7), U14.10 (3B), U4.5 (A7), U5.3 (A7)
- net ADR8: now also U10.25 (A8), U11.27 (A8), U14.12 (4A), U4.27 (A8), U5.25 (A8)
- net ADR9: now also U10.24 (A9), U11.26 (A9), U14.13 (4B), U4.26 (A9), U5.24 (A9)
- net DATA0: now also U10.11 (I/O0), U11.13 (I/O0), U13.3 (D0), U4.13 (I/O0), U7.3 (D0), U8.3 (D0)
- net DATA1: now also U10.12 (I/O1), U11.14 (I/O1), U13.4 (D1), U4.14 (I/O1), U7.4 (D1), U8.4 (D1)
- net DATA2: now also U10.13 (I/O2), U11.15 (I/O2), U13.7 (D2), U4.15 (I/O2), U7.7 (D2), U8.7 (D2)
- net DATA3: now also U10.15 (I/O3), U11.17 (I/O3), U13.8 (D3), U4.17 (I/O3), U7.8 (D3), U8.8 (D3)
- net DATA4: now also U10.16 (I/O4), U11.18 (I/O4), U13.13 (D4), U4.18 (I/O4), U7.13 (D4), U8.13 (D4)
- net DATA5: now also U10.17 (I/O5), U11.19 (I/O5), U13.14 (D5), U4.19 (I/O5), U7.14 (D5), U8.14 (D5)
- net DATA6: now also U10.18 (I/O6), U11.20 (I/O6), U13.17 (D6), U4.20 (I/O6), U7.17 (D6), U8.17 (D6)
- net DATA7: now also U10.19 (I/O7), U11.21 (I/O7), U13.18 (D7), U4.21 (I/O7), U7.18 (D7), U8.18 (D7)
- net GND: now also C1.2, C12.2, C13.2, C15.2, C16.2, C17.2, C18.2, C19.2, C20.2, C21.2, R11.1, R12.1, U10.14 (GND), U11.16 (GND), U12.7 (GND), U13.10 (GND), U14.7 (GND), U15.7 (GND), U16.7 (GND), U17.7 (GND), U18.7 (GND), U4.16 (GND), U5.14 (GND), U5.20 (~{CE}), U7.10 (GND), U8.10 (GND), U9.7 (GND); no longer C1.1, C12.1, C13.1
- net RAM_PAGE_SEL_0: now also U15.9 (3A), U7.2 (O0); no longer U3.31 (A15)
- net RAM_PAGE_SEL_1: now also U15.4 (2A), U7.5 (O1); no longer U3.2 (A16)
- net ~{INT}: now also R16.2
- net ~{I/O_CE}: now also U18.8 (3Y)
- net ~{MREQ}: now also U5.22 (~{OE})
- net ~{RAM_CE}: now also U12.3, U5.13 (I/O2)
- net ~{READ}: now also U10.22 (~{OE}), U11.24 (~{OE}), U4.24 (~{OE})
- net ~{RESET_SIGNAL}: now also U13.1 (~{Mr})
- net ~{WRITE}: now also U12.13
- net PA4: now reaches U2.10 (PA4)
- net PA4: now also J1.5 (Pin_5)
- net PA3: now reaches U2.12 (PA3)
- net PA3: now also J1.4 (Pin_4)
- net PA2: now reaches U2.13 (PA2)
- net PA2: now also J1.3 (Pin_3)
- net PA1: now reaches U2.14 (PA1)
- net PA1: now also J1.2 (Pin_2)
- net PA0: now reaches U2.15 (PA0)
- net PA0: now also J1.1 (Pin_1)
- net ~{ASTB}: now reaches U2.16 (~{ASTB})
- net ~{ASTB}: now also J1.10 (Pin_10)
- net ~{BSTB}: now reaches U2.17 (~{BSTB})
- net ~{BSTB}: now also J2.10 (Pin_10)
- net ARDY: now reaches U2.18 (ARDY)
- net ARDY: now also J1.9 (Pin_9)
- net BRDY: now reaches U2.21 (BRDY)
- net BRDY: now also J2.9 (Pin_9)
- net PB0: now reaches U2.27 (PB0)
- net PB0: now also J2.1 (Pin_1)
- net PB1: now reaches U2.28 (PB1)
- net PB1: now also J2.2 (Pin_2)
- net PB2: now reaches U2.29 (PB2)
- net PB2: now also J2.3 (Pin_3)
- net PB3: now reaches U2.30 (PB3)
- net PB3: now also J2.4 (Pin_4)
- net PB4: now reaches U2.31 (PB4)
- net PB4: now also J2.5 (Pin_5)
- net PB5: now reaches U2.32 (PB5)
- net PB5: now also J2.6 (Pin_6)
- net PB6: now reaches U2.33 (PB6)
- net PB6: now also J2.7 (Pin_7)
- net PB7: now reaches U2.34 (PB7)
- net PB7: now also J2.8 (Pin_8)
- net PA7: now reaches U2.7 (PA7)
- net PA7: now also J1.8 (Pin_8)
- net PA6: now reaches U2.8 (PA6)
- net PA6: now also J1.7 (Pin_7)
- net PA5: now reaches U2.9 (PA5)
- net PA5: now also J1.6 (Pin_6)
- new net: R14.1, U11.31 (~{WE})
- new net: U15.3 (1Y), U3.2 (A16)
- new net: U15.6 (2Y), U3.31 (A15)
- new net: U15.8 (3Y), U3.3 (A14)
- new net: R15.2, U11.1 (~{RESET})
- new net: U16.11 (4Y), U18.4 (2A)
- new net: U16.6 (2Y), U18.1 (1A)
- new net: U16.8 (3Y), U18.2 (1B)
- new net: U13.11 (Cp), U9.8 (3Y)
- new net: R13.1, U10.27 (~{WE})
- new net: R11.2, U8.1 (OE)
- new net: U12.12, U9.1 (1A), U9.4 (2A), U9.9 (3A)
- new net: U12.1, U17.3 (1Y)
- new net: U12.2, U18.5 (2B)
- new net: R12.2, U7.1 (OE)
- new net: U7.11 (Cp), U9.3 (1Y)
- new net: U18.10 (3B), U18.6 (2Y)
- new net: U18.3 (1Y), U18.9 (3A)
- new net: U8.11 (Cp), U9.6 (2Y)
- new net: R9.1, U4.31 (~{WE})
- new net: U12.4, U9.12 (4A)
- new net BIOS_LATCH: U5.18 (I/O6), U9.5 (2B)
- new net BIOS_PAGE_SEL_0: U11.28 (A13), U8.2 (O0)
- new net BIOS_PAGE_SEL_1: U11.29 (A14), U8.5 (O1)
- new net BIOS_PAGE_SEL_2: U11.3 (A15), U8.6 (O2)
- new net BIOS_PAGE_SEL_3: U11.2 (A16), U8.9 (O3)
- new net BIOS_PAGE_SEL_4: U11.30 (A17), U8.12 (O4)
- new net FLASH_PAGE_SEL_0: U4.29 (A14), U7.9 (O3)
- new net FLASH_PAGE_SEL_1: U4.3 (A15), U7.12 (O4)
- new net FLASH_PAGE_SEL_2: U4.2 (A16), U7.15 (O5)
- new net FLASH_PAGE_SEL_3: U4.30 (A17), U7.16 (O6)
- new net FLASH_PAGE_SEL_4: U4.1 (A18), U7.19 (O7)
- new net IO_SEL_1: U14.3 (1Y), U16.4 (2A)
- new net IO_SEL_2: U14.6 (2Y), U16.5 (2B)
- new net IO_SEL_3: U14.8 (3Y), U16.9 (3A)
- new net IO_SEL_4: U14.11 (4Y), U16.10 (3B)
- new net IO_SEL_5: U16.12 (4A), U16.3 (1Y)
- new net IO_SEL_6: U16.13 (4B), U18.11 (4Y)
- new net OUTPUT_LATCH: U5.19 (I/O7), U9.10 (3B)
- new net RAM_PAGE_SEL_2: U15.1 (1A), U7.6 (O2)
- new net RAM_PAGE_SEL_OVERRIDE: U15.10 (3B), U15.2 (1B), U15.5 (2B), U9.11 (4Y)
- new net RAM/FLASH_LATCH: U5.17 (I/O5), U9.2 (1B)
- new net ~{BIOS_CE}: U11.22 (~{CE}), U5.12 (I/O1)
- new net ~{BIOS_MAIN_CE}: U10.20 (~{CE}), U5.11 (I/O0)
- new net ~{FLASH_CE}: U4.22 (~{CE}), U5.15 (I/O3)
Other:
- note added: "1100 0000 0000 00XX"
- note added: "20 LED + 5 LED + 4 LED"
- note added: "ADDRESS SPACE (64kB, divided into 4 main 16kB segments) 0000 - 3FFF EEPROM BIOS 0000 - 1FFF BIOS MAIN 2000 - 3FFF BIOS PAGED (32 pages, 256kB total memory) 4000 - 7FFF RAM (8 pages, 128kB total memory) 8000 - BFFF FLASH program memory (32 pages, 512kB total memory) C000 - FFFF Misc (I/O, page switching) + LAST 8kB OF RAM (ALWAYS AVAILABLE) I/O chip: C000 Port A, Data C001 Port B, Data C002 Port A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"
- note added: "BIOS"
- note added: "EN29F040 - 512kB FLASH TC551001CP - 128kB RAM W49F002 - 256kB PAGED BIOS AT28C64 - 16kB MAIN BIOS W27E512 - 64kB CHIP SELECT"
- note added: "RAM/FLASH"
- note removed: "ADDRESS DECODE"
- note removed: "ADDRESS SPACE (64kB, podzielone na 16kB segmenty) 0000 - 3FFF EEPROM 0000 - 1FFF EEPROM BIOS 2000 - 3FFF EEPROM wymienny 4000 - 7FFFF I/O + paging RAMu (Adresy dalej podzielone na 4 multiplekserem (4kB)) I/O chip: 4000 Port A, Data 4001 Port B, Data 4002 Port A, Command 4003 Port B, Command RAM paging (D flip-flop) strona ustawiana adresem, zegar wywołany linią danych (DATA 0) po wybraniu adresów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"
- note removed: "ADDRESS SPACE SIGNAL"
- moved on the sheet: C11, C14, C2, C3, C4, C5, C6, C7, C8, R1, R10, R2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

Commit message: updatus
Other:
- note added: "20 LED I/O"
- note removed: "20 LED + 5 LED + 4 LED"
- moved on the sheet: U12C, U12D, U12E
Changed lines of the file:
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@@
 		)
 	)
-	(text "20 LED\n+ 5 LED\n+ 4 LED"
+	(text "20 LED I/O\n"
 		(exclude_from_sim no)
 		(at 534.416 57.15 0)
@@
 	(symbol
 		(lib_id "74xx:74HC14")
-		(at 227.33 312.42 0)
+		(at 514.35 156.21 0)
 		(unit 3)
 		(exclude_from_sim no)
@@
 		(fields_autoplaced yes)
 		(property "Reference" "U12"
-			(at 227.33 303.53 0)
+			(at 514.35 147.32 0)
 			(effects
 				(font
@@
 		)
 		(property "Value" "74HC14"
-			(at 227.33 306.07 0)
+			(at 514.35 149.86 0)
 			(effects
 				(font
@@
 		)
 		(property "Footprint" "Package_SO:SO-14_3.9x8.65mm_P1.27mm"
-			(at 227.33 312.42 0)
+			(at 514.35 156.21 0)
 			(effects
 				(font
@@
 		)
 		(property "Datasheet" "http://www.ti.com/lit/gpn/sn74HC14"
-			(at 227.33 312.42 0)
+			(at 514.35 156.21 0)
 			(effects
 				(font
@@
 		)
 		(property "Description" "Hex inverter schmitt trigger"
-			(at 227.33 312.42 0)
+			(at 514.35 156.21 0)
 			(effects
 				(font
@@
 	(symbol
 		(lib_id "74xx:74HC14")
-		(at 278.13 309.88 0)
+		(at 565.15 153.67 0)
 		(unit 5)
 		(exclude_from_sim no)
@@
 		(fields_autoplaced yes)
 		(property "Reference" "U12"
-			(at 278.13 300.99 0)
+			(at 565.15 144.78 0)
 			(effects
 				(font
@@
 		)
 		(property "Value" "74HC14"
-			(at 278.13 303.53 0)
+			(at 565.15 147.32 0)
 			(effects
 				(font
@@
 		)
 		(property "Footprint" "Package_SO:SO-14_3.9x8.65mm_P1.27mm"
-			(at 278.13 309.88 0)
+			(at 565.15 153.67 0)
 			(effects
 				(font
@@
 		)
 		(property "Datasheet" "http://www.ti.com/lit/gpn/sn74HC14"
-			(at 278.13 309.88 0)
+			(at 565.15 153.67 0)
 			(effects
 				(font
@@
 		)
 		(property "Description" "Hex inverter schmitt trigger"
-			(at 278.13 309.88 0)
+			(at 565.15 153.67 0)
 			(effects
 				(font
@@
 	(symbol
 		(lib_id "74xx:74HC14")
-		(at 252.73 311.15 0)
+		(at 539.75 154.94 0)
 		(unit 4)
 		(exclude_from_sim no)
@@
 		(fields_autoplaced yes)
 		(property "Reference" "U12"
-			(at 252.73 302.26 0)
+			(at 539.75 146.05 0)
 			(effects
 				(font
@@
 		)
 		(property "Value" "74HC14"
-			(at 252.73 304.8 0)
+			(at 539.75 148.59 0)
 			(effects
 				(font
@@
 		)
 		(property "Footprint" "Package_SO:SO-14_3.9x8.65mm_P1.27mm"
-			(at 252.73 311.15 0)
+			(at 539.75 154.94 0)
 			(effects
 				(font
@@
 		)
 		(property "Datasheet" "http://www.ti.com/lit/gpn/sn74HC14"
-			(at 252.73 311.15 0)
+			(at 539.75 154.94 0)
 			(effects
 				(font
@@
 		)
 		(property "Description" "Hex inverter schmitt trigger"
-			(at 252.73 311.15 0)
+			(at 539.75 154.94 0)
 			(effects
 				(font

Commit message: sdfsdf
Parts:
- added C22, C23, C24: 100n, symbol Device:C
- added D1, D10, D11, D12, D2, D3, D4, D5, D6, D7, D8, D9: LED, symbol Device:LED
- added R17, R18, R19, R20, R21, R22, R23, R24, R25, R26, R27, R28: 1k, symbol Device:R
- added U19, U20, U21: SN74AC00N, N14, symbol Custom_symbole:SN74AC00N
Connections:
- net +5V: now also C22.1, C23.1, C24.1, R17.2, R18.2, R19.2, R20.2, R21.2, R22.2, R23.2, R24.2, U19.14 (VCC), U20.14 (VCC), U21.14 (VCC)
- net DATA0: now also U19.1 (1A), U19.2 (1B)
- net DATA1: now also U19.4 (2A), U19.5 (2B)
- net DATA2: now also U19.10 (3B), U19.9 (3A)
- net DATA3: now also U19.12 (4A), U19.13 (4B)
- net DATA4: now also U20.1 (1A), U20.2 (1B)
- net DATA5: now also U20.4 (2A), U20.5 (2B)
- net DATA6: now also U20.10 (3B), U20.9 (3A)
- net DATA7: now also U20.12 (4A), U20.13 (4B)
- net GND: now also C22.2, C23.2, C24.2, R25.2, R26.2, R27.2, R28.2, U19.7 (GND), U20.7 (GND), U21.7 (GND)
- net ~{IORQ}: now also U21.12 (4A), U21.13 (4B)
- net ~{I/O_CE}: now also U5.16 (I/O4)
- net ~{MREQ}: now also U21.10 (3B), U21.9 (3A)
- net ~{READ}: now also U21.1 (1A), U21.2 (1B)
- net ~{WRITE}: now also U21.4 (2A), U21.5 (2B)
- new net: D12.1 (K), R28.1
- new net: D8.1 (K), U20.11 (4Y)
- new net: D8.2 (A), R24.1
- new net: D5.1 (K), U20.3 (1Y)
- new net: D5.2 (A), R21.1
- new net: D3.2 (A), R19.1
- new net: D2.1 (K), U19.6 (2Y)
- new net: D2.2 (A), R18.1
- new net: D4.2 (A), R20.1
- new net: D10.1 (K), R26.1
- new net: D9.1 (K), R25.1
- new net: D9.2 (A), U21.3 (1Y)
- new net: D3.1 (K), U19.8 (3Y)
- new net: D7.2 (A), R23.1
- new net: D4.1 (K), U19.11 (4Y)
- new net: D1.1 (K), U19.3 (1Y)
- new net: D12.2 (A), U21.11 (4Y)
- new net: D10.2 (A), U21.6 (2Y)
- new net: D11.2 (A), U21.8 (3Y)
- new net: D11.1 (K), R27.1
- new net: D6.1 (K), U20.6 (2Y)
- new net: D7.1 (K), U20.8 (3Y)
- new net: D6.2 (A), R22.1
- new net: D1.2 (A), R17.1
Other:
- moved on the sheet: C15, C7, J1, J2, R10, R16, U12B, U12F, U12G, U2

Commit message: adasd
Parts:
- removed C22, C23, C24: 100n, symbol Device:C
- removed D1, D10, D11, D12, D2, D3, D4, D5, D6, D7, D8, D9: LED, symbol Device:LED
- removed R17, R18, R19, R20, R21, R22, R23, R24, R25, R26, R27, R28: 1k, symbol Device:R
- removed U19, U20, U21: SN74AC00N, N14, symbol Custom_symbole:SN74AC00N
- added J3: Conn_01x08_Socket, Connector_PinSocket_2.54mm:PinSocket_1x08_P2.54mm_Vertical, symbol Connector:Conn_01x08_Socket
- added J4: Conn_01x03_Socket, Connector_PinSocket_2.54mm:PinSocket_1x03_P2.54mm_Vertical, symbol Connector:Conn_01x03_Socket
Connections:
- net ADR15: now also U17.5 (2B); no longer U9.13 (4B)
- net RAM_PAGE_SEL_OVERRIDE: now also U17.6 (2Y); no longer U9.11 (4Y)
- net ~{I/O_CE}: no longer U5.16 (I/O4)
- net at U13.12 (Q4): now also J3.5 (Pin_5)
- net at U13.15 (Q5): now also J3.6 (Pin_6)
- net at U13.16 (Q6): now also J3.7 (Pin_7)
- net at U13.19 (Q7): now also J3.8 (Pin_8)
- net at U13.2 (Q0): now also J3.1 (Pin_1)
- net at U13.5 (Q1): now also J3.2 (Pin_2)
- net at U13.6 (Q2): now also J3.3 (Pin_3)
- net at U13.9 (Q3): now also J3.4 (Pin_4)
- net at U8.15 (O5): now also J4.1 (Pin_1)
- net at U8.16 (O6): now also J4.2 (Pin_2)
- net at U8.19 (O7): now also J4.3 (Pin_3)
- net at U17.4 (2A): now also U12.4
- net at U9.12 (4A): no longer U12.4
Other:
- moved on the sheet: C18, C19, C20, C21, U12A, U12C, U12D, U12E, U14, U16, U17, U18

Commit message: asdas
Parts:
- added D1, D10, D11, D12, D13, D14, D15, D16, D17, D3, D4, D5, D6, D7, D8, D9: LED_WHITE, symbol Device:LED
- added D18, D19, D20, D21, D22, D23, D24, D25: LED_YELLOW, symbol Device:LED
- added D2: LED, symbol Device:LED
- added Q1, Q10, Q11, Q12, Q13, Q14, Q15, Q16, Q17, Q18, Q19, Q20, Q21, Q22, Q23, Q24, Q25, Q3, Q4, Q5, Q6, Q7, Q8, Q9: NMOS, Package_TO_SOT_THT:TO-92, symbol Simulation_SPICE:NMOS
- added Q2: PMOS, Package_TO_SOT_THT:TO-92, symbol Simulation_SPICE:PMOS
- added R17, R18, R19, R20, R21, R22, R23, R24, R25, R26, R27, R28, R29, R30, R31, R32, R33, R34, R35, R36, R37, R38, R39, R40, R41: 1k, symbol Device:R
- C2: value C -> 100n
- C4: value C -> 10n
- R2: value R -> 1M
- R4: value R -> 1k
- SW1: value SW_Push -> RESET
- SW2: value SW_Push -> CLK_STEP
Connections:
- net +5V: now also R17.1, R18.1, R19.1, R20.1, R21.1, R22.1, R23.1, R24.1, R25.1, R26.1, R27.1, R28.1, R29.1, R30.1, R31.1, R32.1, R33.1, R34.1, R35.1, R36.1, R37.1, R38.1, R39.1, R40.1, R41.1
- net ADR0: now also Q1.2 (G)
- net ADR1: now also Q3.2 (G)
- net ADR10: now also Q8.2 (G)
- net ADR11: now also Q9.2 (G)
- net ADR12: now also Q11.2 (G)
- net ADR13: now also Q13.2 (G)
- net ADR14: now also Q15.2 (G)
- net ADR15: now also Q17.2 (G)
- net ADR2: now also Q4.2 (G)
- net ADR3: now also Q5.2 (G)
- net ADR4: now also Q10.2 (G)
- net ADR5: now also Q12.2 (G)
- net ADR6: now also Q14.2 (G)
- net ADR7: now also Q16.2 (G)
- net ADR8: now also Q6.2 (G)
- net ADR9: now also Q7.2 (G)
- net DATA0: now also Q18.2 (G)
- net DATA1: now also Q20.2 (G)
- net DATA2: now also Q22.2 (G)
- net DATA3: now also Q24.2 (G)
- net DATA4: now also Q19.2 (G)
- net DATA5: now also Q21.2 (G)
- net DATA6: now also Q23.2 (G)
- net DATA7: now also Q25.2 (G)
- net GND: now also Q1.3 (S), Q10.3 (S), Q11.3 (S), Q12.3 (S), Q13.3 (S), Q14.3 (S), Q15.3 (S), Q16.3 (S), Q17.3 (S), Q18.3 (S), Q19.3 (S), Q2.1 (D), Q20.3 (S), Q21.3 (S), Q22.3 (S), Q23.3 (S), Q24.3 (S), Q25.3 (S), Q3.3 (S), Q4.3 (S), Q5.3 (S), Q6.3 (S), Q7.3 (S), Q8.3 (S), Q9.3 (S)
- new net: D1.1 (K), Q1.1 (D)
- new net: D1.2 (A), R17.2
- new net: D17.1 (K), Q17.1 (D)
- new net: D17.2 (A), R33.2
- new net: D16.1 (K), Q16.1 (D)
- new net: D16.2 (A), R32.2
- new net: D6.2 (A), R22.2
- new net: D23.1 (K), Q23.1 (D)
- new net: D23.2 (A), R39.2
- new net: D8.1 (K), Q8.1 (D)
- new net: D13.1 (K), Q13.1 (D)
- new net: D13.2 (A), R29.2
- new net: D3.1 (K), Q3.1 (D)
- new net: D10.1 (K), Q10.1 (D)
- new net: D10.2 (A), R26.2
- new net: D21.2 (A), R37.2
- new net: D19.1 (K), Q19.1 (D)
- new net: D19.2 (A), R35.2
- new net: D20.1 (K), Q20.1 (D)
- new net: D20.2 (A), R36.2
- new net: D15.1 (K), Q15.1 (D)
- new net: D11.1 (K), Q11.1 (D)
- new net: D11.2 (A), R27.2
- new net: D7.2 (A), R23.2
- new net: D9.1 (K), Q9.1 (D)
- new net: D9.2 (A), R25.2
- new net: D7.1 (K), Q7.1 (D)
- new net: D18.2 (A), R34.2
- new net: D12.1 (K), Q12.1 (D)
- new net: D22.1 (K), Q22.1 (D)
- new net: D22.2 (A), R38.2
- new net: D21.1 (K), Q21.1 (D)
- new net: D24.1 (K), Q24.1 (D)
- new net: D15.2 (A), R31.2
- new net: D14.1 (K), Q14.1 (D)
- new net: D14.2 (A), R30.2
- new net: D18.1 (K), Q18.1 (D)
- new net: D4.2 (A), R20.2
- new net: D12.2 (A), R28.2
- new net: D8.2 (A), R24.2
- new net: D2.1 (K), Q2.3 (S)
- new net: D6.1 (K), Q6.1 (D)
- new net: D5.1 (K), Q5.1 (D)
- new net: D24.2 (A), R40.2
- new net: D5.2 (A), R21.2
- new net: D25.1 (K), Q25.1 (D)
- new net: D4.1 (K), Q4.1 (D)
- new net: D25.2 (A), R41.2
- new net: D2.2 (A), R18.2
- new net: D3.2 (A), R19.2
