File: z80_schematic.kicad_sch (KiCad schematic)
At the start: 136 parts, among them J1 Port_A, J2 Port_B, J3 Conn_01x08_Socket, J4 Conn_01x03_Socket, Q1 NMOS, Q10 NMOS, Q11 NMOS, Q12 NMOS, Q13 NMOS, Q14 NMOS, Q15 NMOS, Q16 NMOS, Q17 NMOS, Q18 NMOS, Q19 NMOS, Q2 PMOS, Q20 NMOS, Q21 NMOS, Q22 NMOS, Q23 NMOS, Q24 NMOS, Q25 NMOS, Q3 NMOS, Q4 NMOS, Q5 NMOS, Q6 NMOS, Q7 NMOS, Q8 NMOS, Q9 NMOS, SW1 RESET, SW2 CLK_STEP, U1 Z80CPU, U10 AT28C64B-15PU, U11 W49F002, U12 74HC14, U13 74HCT273, U14 SN74AC32, U15 SN74AC32, U16 SN74AC32, U17 SN74ACT08N, U18 SN74AC32, U2 Z84C20, U3 TC551001CP-70L, U4 EN29F040A, U5 W27E512, U6 NE555P, U7 74HC374, U8 74HC374, U9 SN74ACT08N

Commit message: dfg
Parts:
- removed D18, D19, D20, D21, D22, D23, D24, D25: LED_YELLOW, symbol Device:LED
- removed D2: LED, symbol Device:LED
- removed Q1, Q10, Q11, Q12, Q13, Q24, Q25, Q3, Q4, Q5, Q6, Q7, Q8, Q9: NMOS, Package_TO_SOT_THT:TO-92, symbol Simulation_SPICE:NMOS
- removed Q2: PMOS, Package_TO_SOT_THT:TO-92, symbol Simulation_SPICE:PMOS
- removed R40, R41: 1k, symbol Device:R
- added Q1, Q10, Q11, Q12, Q13, Q3, Q4, Q5, Q6, Q7, Q8, Q9: PMOS, Package_TO_SOT_THT:TO-92, symbol Simulation_SPICE:PMOS
- added Q2: NMOS, Package_TO_SOT_THT:TO-92, symbol Simulation_SPICE:NMOS
- added U19: 27C512, Package_DIP:DIP-28_W15.24mm_Socket_LongPads, symbol Memory_EPROM:27C512
- added U25, U26: D148K, Display_7Segment:D1X8K, symbol Display_Character:D148K
- D1, D10, D11, D12, D13, D3, D4, D5, D6, D7, D8, D9: value LED_WHITE -> LED
- D14, D15, D16, D17: value LED_WHITE -> LED_YELLOW
Connections:
- net +5V: now also Q1.3 (S), Q10.3 (S), Q11.3 (S), Q12.3 (S), Q13.3 (S), Q3.3 (S), Q4.3 (S), Q5.3 (S), Q6.3 (S), Q7.3 (S), Q8.3 (S), Q9.3 (S); no longer R17.1, R18.1, R19.1, R20.1, R21.1, R22.1, R23.1, R24.1, R25.1, R26.1, R27.1, R28.1, R29.1, R34.1, R35.1, R36.1, R37.1, R38.1, R39.1
- net ADR14: no longer Q15.2 (G)
- net ADR15: no longer Q17.2 (G)
- net ADR6: no longer Q14.2 (G)
- net ADR7: no longer Q16.2 (G)
- net BIOS_LATCH: now also Q15.2 (G)
- net CLK: now also Q17.2 (G)
- net DATA0: no longer Q18.2 (G)
- net DATA1: no longer Q20.2 (G)
- net DATA2: no longer Q22.2 (G)
- net DATA4: no longer Q19.2 (G)
- net DATA5: no longer Q21.2 (G)
- net DATA6: no longer Q23.2 (G)
- net GND: now also R17.1, R19.1, R20.1, R21.1, R22.1, R23.1, R24.1, R25.1, R26.1, R27.1, R28.1, R29.1, Q2.3 (S)
- net OUTPUT_LATCH: now also Q14.2 (G)
- net RAM/FLASH_LATCH: now also Q16.2 (G)
- net ~{BIOS_CE}: now also Q11.2 (G)
- net ~{BIOS_MAIN_CE}: now also Q10.2 (G)
- net ~{FLASH_CE}: now also Q13.2 (G)
- net ~{INT}: now also Q7.2 (G)
- net ~{IORQ}: now also Q5.2 (G)
- net ~{I/O_CE}: now also Q9.2 (G)
- net ~{M1}: now also Q6.2 (G)
- net ~{MREQ}: now also Q4.2 (G)
- net ~{RAM_CE}: now also Q12.2 (G)
- net ~{READ}: now also Q1.2 (G)
- net ~{RESET_SIGNAL}: now also Q8.2 (G)
- net ~{WRITE}: now also Q3.2 (G)
- net at D1.1 (K): now also R17.2
- net at D1.2 (A): now also Q1.1 (D); no longer R17.2
- net at R22.2: now also D6.1 (K); no longer D6.2 (A)
- net at Q23.1 (D): now also R39.1
- net at R39.2: now also U25.9 (F), U26.9 (F)
- net at D8.1 (K): now also R24.2
- net at D13.1 (K): now also R29.2
- net at D13.2 (A): now also Q13.1 (D); no longer R29.2
- net at D3.1 (K): now also R19.2
- net at D10.1 (K): now also R26.2
- net at D10.2 (A): now also Q10.1 (D); no longer R26.2
- net at R37.2: now also U25.6 (B), U26.6 (B)
- net at Q19.1 (D): now also R35.1
- net at R35.2: now also U25.1 (E), U26.1 (E)
- net at Q20.1 (D): now also R36.1
- net at R36.2: now also U25.10 (G), U26.10 (G)
- net at D11.1 (K): now also R27.2
- net at D11.2 (A): now also Q11.1 (D); no longer R27.2
- net at R23.2: now also D7.1 (K); no longer D7.2 (A)
- net at D9.1 (K): now also R25.2
- net at D9.2 (A): now also Q9.1 (D); no longer R25.2
- net at R34.2: now also U25.4 (C), U26.4 (C)
- net at D12.1 (K): now also R28.2
- net at Q22.1 (D): now also R38.1
- net at R38.2: now also U25.2 (D), U26.2 (D)
- net at Q21.1 (D): now also R37.1
- net at Q18.1 (D): now also R18.1
- net at R20.2: now also D4.1 (K); no longer D4.2 (A)
- net at D12.2 (A): now also Q12.1 (D); no longer R28.2
- net at D8.2 (A): now also Q8.1 (D); no longer R24.2
- net at D5.1 (K): now also R21.2
- net at D5.2 (A): now also Q5.1 (D); no longer R21.2
- net at R18.2: now also U25.7 (A), U26.7 (A)
- net at D3.2 (A): now also Q3.1 (D); no longer R19.2
- new net: Q18.2 (G), U19.11 (D0)
- new net: D6.2 (A), Q6.1 (D)
- new net: Q2.1 (D), R34.1
- new net: Q2.2 (G), U19.13 (D2)
- new net: Q20.2 (G), U19.18 (D6)
- new net: Q21.2 (G), U19.12 (D1)
- new net: D4.2 (A), Q4.1 (D)
- new net: Q19.2 (G), U19.16 (D4)
- new net: Q22.2 (G), U19.15 (D3)
- new net: Q23.2 (G), U19.17 (D5)
- new net: D7.2 (A), Q7.1 (D)
Other:
- moved on the sheet: C1, C10, C12, C13, C14, C15, C16, C17, C18, C19, C20, C21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
