File: z80_schematic.kicad_sch (KiCad schematic)
At the start: 126 parts, among them J1 Port_A, J2 Port_B, J3 Conn_01x08_Socket, J4 Conn_01x03_Socket, Q1 PMOS, Q10 PMOS, Q11 PMOS, Q12 PMOS, Q13 PMOS, Q14 NMOS, Q15 NMOS, Q16 NMOS, Q17 NMOS, Q18 NMOS, Q19 NMOS, Q2 NMOS, Q20 NMOS, Q21 NMOS, Q22 NMOS, Q23 NMOS, Q3 PMOS, Q4 PMOS, Q5 PMOS, Q6 PMOS, Q7 PMOS, Q8 PMOS, Q9 PMOS, SW1 RESET, SW2 CLK_STEP, U1 Z80CPU, U10 AT28C64B-15PU, U11 W49F002, U12 74HC14, U13 74HCT273, U14 SN74AC32, U15 SN74AC32, U16 SN74AC32, U17 SN74ACT08N, U18 SN74AC32, U19 27C512, U2 Z84C20, U25 D148K, U26 D148K, U3 TC551001CP-70L, U4 EN29F040A, U5 W27E512, U6 NE555P, U7 74HC374, U8 74HC374, U9 SN74ACT08N

Commit message: started decoding and keyboard
Parts:
- removed Q18, Q19, Q2, Q20, Q21, Q22, Q23: NMOS, Package_TO_SOT_THT:TO-92, symbol Simulation_SPICE:NMOS
- added C22, C23, C24, C25, C26, C27: 100n, symbol Device:C
- added Q18, Q19, Q2, Q20, Q21, Q22, Q23, Q26, Q27, Q28, Q29, Q30, Q32, Q33, Q34, Q35, Q37, Q38, Q39, Q40, Q42, Q43, Q44, Q45: PMOS, Package_TO_SOT_THT:TO-92, symbol Simulation_SPICE:PMOS
- added Q24, Q25, Q31, Q36, Q41, Q46: NMOS, Package_TO_SOT_THT:TO-92, symbol Simulation_SPICE:NMOS
- added R40, R47, R55: 10k, symbol Device:R
- added R41, R42, R43, R44, R45, R46, R48, R49, R50, R51, R52, R53, R54, R56: 1k, symbol Device:R
- added U20: 74HC164, Package_DIP:DIP-14_W7.62mm_Socket_LongPads, symbol 74xx:74HC164
- added U21, U23, U24, U28: D148K, Display_7Segment:D1X8K, symbol Display_Character:D148K
- added U22, U27: 27C512, Package_DIP:DIP-28_W15.24mm_Socket_LongPads, symbol Memory_EPROM:27C512
- added U29, U30: SN74ACT08N, Package_DIP:DIP-14_W7.62mm_Socket_LongPads, symbol Custom_symbole:SN74ACT08N
Connections:
- net +5V: now also U19.28 (VCC), C22.1, C23.1, C24.1, C25.1, C26.1, C27.1, Q18.3 (S), Q19.3 (S), Q2.3 (S), Q20.3 (S), Q21.3 (S), Q22.3 (S), Q23.3 (S), Q26.3 (S), Q27.3 (S), Q28.3 (S), Q29.3 (S), Q30.3 (S), Q32.3 (S), Q33.3 (S), Q34.3 (S), Q35.3 (S), Q37.3 (S), Q38.3 (S), Q39.3 (S), Q40.3 (S), Q42.3 (S), Q43.3 (S), Q44.3 (S), Q45.3 (S), U20.14 (VCC), U22.28 (VCC), U27.28 (VCC), U29.14 (VDD), U30.14 (VDD)
- net ADR0: now also U19.10 (A0)
- net ADR1: now also U19.9 (A1)
- net ADR10: now also U22.8 (A2)
- net ADR11: now also U22.7 (A3)
- net ADR12: now also U22.6 (A4)
- net ADR13: now also U22.5 (A5)
- net ADR14: now also U22.4 (A6)
- net ADR15: now also U22.3 (A7)
- net ADR2: now also U19.8 (A2)
- net ADR3: now also U19.7 (A3)
- net ADR4: now also U19.6 (A4)
- net ADR5: now also U19.5 (A5)
- net ADR6: now also U19.4 (A6)
- net ADR7: now also U19.3 (A7)
- net ADR8: now also U22.10 (A0)
- net ADR9: now also U22.9 (A1)
- net DATA0: now also U27.10 (A0), U29.3 (1Y)
- net DATA1: now also U27.9 (A1), U29.6 (2Y)
- net DATA2: now also U27.8 (A2), U29.8 (3Y)
- net DATA3: now also U27.7 (A3), U29.11 (4Y)
- net DATA4: now also U27.6 (A4), U30.3 (1Y)
- net DATA5: now also U27.5 (A5), U30.6 (2Y)
- net DATA6: now also U27.4 (A6), U30.8 (3Y)
- net DATA7: now also U27.3 (A7), U30.11 (4Y)
- net GND: now also U19.1 (A15), U19.14 (GND), U19.2 (A12), U19.21 (A10), U19.23 (A11), U19.24 (A9), U19.26 (A13), U19.27 (A14), C22.2, C23.2, C24.2, C25.2, C26.2, C27.2, Q24.3 (S), Q25.3 (S), Q31.3 (S), Q36.3 (S), Q41.3 (S), Q46.3 (S), R40.1, R47.1, R55.1, U20.7 (GND), U22.1 (A15), U22.14 (GND), U22.2 (A12), U22.21 (A10), U22.23 (A11), U22.24 (A9), U22.26 (A13), U22.27 (A14), U27.1 (A15), U27.14 (GND), U27.2 (A12), U27.21 (A10), U27.23 (A11), U27.24 (A9), U27.26 (A13), U27.27 (A14), U29.7 (GND), U30.7 (GND)
- net ~{READ}: now also U12.5
- net at U25.1 (E), U26.1 (E): now also R37.2; no longer R35.2
- net at U25.10 (G), U26.10 (G): now also R39.2; no longer R36.2
- net at U25.2 (D), U26.2 (D): now also R36.2; no longer R38.2
- net at U25.3 (CC): now also U25.8 (CC), Q25.1 (D)
- net at U25.4 (C), U26.4 (C): now also R35.2; no longer R34.2
- net at U25.6 (B), U26.6 (B): now also R34.2; no longer R37.2
- net at U25.9 (F), U26.9 (F): now also R38.2; no longer R39.2
- net at R18.1: now also Q18.1 (D)
- net at U19.11 (D0): now also Q18.2 (G)
- net at U12.6: now also U9.13 (4B)
- net at R34.1: now also Q2.1 (D)
- net at U19.13 (D2): now also Q19.2 (G)
- net at R38.1: now also Q22.1 (D)
- net at R36.1: now also Q20.1 (D)
- net at U19.18 (D6): now also Q23.2 (G)
- net at R37.1: now also Q21.1 (D)
- net at U19.12 (D1): now also Q2.2 (G)
- net at R39.1: now also Q23.1 (D)
- net at R35.1: now also Q19.1 (D)
- net at U19.16 (D4): now also Q21.2 (G)
- net at U19.15 (D3): now also Q20.2 (G)
- net at U19.17 (D5): now also Q22.2 (G)
- net at U19.19 (D7): now also Q25.2 (G), Q26.2 (G)
- net 200Hz_CLK: now reaches U19.25 (A8)
- net 200Hz_CLK: now also U22.25 (A8), U27.25 (A8)
- net KEYBOARD: now reaches U5.16 (I/O4)
- net KEYBOARD: now also U9.12 (4A)
- net at U26.3 (CC): now also U26.8 (CC), Q24.1 (D)
- net at U9.11 (4Y): now also U29.10 (3B), U29.13 (4B), U29.2 (1B), U29.5 (2B), U30.10 (3B), U30.13 (4B), U30.2 (1B), U30.5 (2B)
- net OUTPUT_LATCH renamed DISPLAY
- new net: U20.10 (Q4), U30.1 (1A)
- new net: U20.11 (Q5), U30.4 (2A)
- new net: U20.12 (Q6), U30.9 (3A)
- new net: U20.13 (Q7), U30.12 (4A)
- new net: U20.3 (Q0), U29.1 (1A)
- new net: U20.4 (Q1), U29.4 (2A)
- new net: U20.5 (Q2), U29.9 (3A)
- new net: U20.6 (Q3), U29.12 (4A)
- new net: Q29.1 (D), Q31.2 (G), R47.2
- new net: Q46.1 (D), U28.3 (CC), U28.8 (CC)
- new net: Q39.2 (G), Q46.2 (G), U27.19 (D7)
- new net: Q28.1 (D), R42.1
- new net: Q28.2 (G), U22.12 (D1)
- new net: Q29.2 (G), Q36.2 (G), U22.19 (D7)
- new net: Q31.1 (D), U21.3 (CC), U21.8 (CC)
- new net: R53.2, U24.1 (E), U28.1 (E)
- new net: R56.2, U24.10 (G), U28.10 (G)
- new net: R52.2, U24.2 (D), U28.2 (D)
- new net: Q41.1 (D), U24.3 (CC), U24.8 (CC)
- new net: R51.2, U24.4 (C), U28.4 (C)
- new net: R50.2, U24.6 (B), U28.6 (B)
- new net: R49.2, U24.7 (A), U28.7 (A)
- new net: R54.2, U24.9 (F), U28.9 (F)
- new net: Q27.2 (G), U22.11 (D0)
- new net: Q30.2 (G), U22.13 (D2)
- new net: Q32.2 (G), U22.15 (D3)
- new net: Q33.2 (G), U22.16 (D4)
- new net: Q34.2 (G), U22.17 (D5)
- new net: Q35.2 (G), U22.18 (D6)
- new net: Q38.1 (D), R50.1
- new net: Q38.2 (G), U27.12 (D1)
- new net: Q45.1 (D), R56.1
- new net: Q45.2 (G), U27.18 (D6)
- new net: Q39.1 (D), Q41.2 (G), R55.2
- new net: Q24.2 (G), Q26.1 (D), R40.2
- new net: Q44.1 (D), R54.1
- new net: Q35.1 (D), R48.1
- new net: R48.2, U21.10 (G), U23.10 (G)
- new net: R42.2, U21.6 (B), U23.6 (B)
- new net: Q44.2 (G), U27.17 (D5)
- new net: Q37.1 (D), R49.1
- new net: Q34.1 (D), R46.1
- new net: R46.2, U21.9 (F), U23.9 (F)
- new net: Q36.1 (D), U23.3 (CC), U23.8 (CC)
- new net: Q42.1 (D), R52.1
- new net: Q43.1 (D), R53.1
- new net: Q37.2 (G), U27.11 (D0)
- new net: Q40.2 (G), U27.13 (D2)
- new net: Q42.2 (G), U27.15 (D3)
- new net: Q43.2 (G), U27.16 (D4)
- new net: Q33.1 (D), R45.1
- new net: Q27.1 (D), R41.1
- new net: Q40.1 (D), R51.1
- new net: Q30.1 (D), R43.1
- new net: R43.2, U21.4 (C), U23.4 (C)
- new net: R41.2, U21.7 (A), U23.7 (A)
- new net: Q32.1 (D), R44.1
- new net: R45.2, U21.1 (E), U23.1 (E)
- new net: R44.2, U21.2 (D), U23.2 (D)
Other:
- note added: "ADDR 0 - 7 hex decoding"
- note added: "ADDR 8 - 15 hex decoding"
- note added: "Address decoding"
- note added: "DATA 0 - 7 hex decoding"
- note added: "Debounced CLK step button"
- note added: "Debounced reset button"
- note added: "FLASH"
- note added: "I/O chip"
- note added: "I/O_CE address decoding"
- note added: "Interrupt line pullup"
- note added: "LCD display output"
- note added: "MAIN BIOS"
- note added: "PAGED BIOS"
- note added: "PS/2 keyboard input with interrupt"
- note added: "RAM"
- note added: "SCHMITT power supply"
- note added: "Signal lines indicators"
- note added: "template"
- note removed: "1100 0000 0000 00XX"
- note removed: "20 LED I/O"
- moved on the sheet: C1, C10, C12, C13, C14, C16, C17, C18, C19, C20, C21, C5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

Commit message: asdsa
Parts:
- removed U29, U30: SN74ACT08N, Package_DIP:DIP-14_W7.62mm_Socket_LongPads, symbol Custom_symbole:SN74ACT08N
- added C28: 100n, symbol Device:C
- added D2: D, symbol Device:D
- added J5: KB_conn, symbol Connector:Conn_01x06_Socket
- added Q47: NMOS, Package_TO_SOT_THT:TO-92, symbol Simulation_SPICE:NMOS
- added R57: 47k, symbol Device:R
- added R58: 10k, symbol Device:R
- added U29: 74HCT374, Package_DIP:DIP-20_W7.62mm_Socket_LongPads, symbol 74xx:74HCT374
- added U30: 74HC164, Package_DIP:DIP-14_W7.62mm_Socket_LongPads, symbol 74xx:74HC164
- C27: value 100n -> 10n
Connections:
- net +5V: now also C28.1, J5.4 (Pin_4), R58.1, U29.20 (VCC), U30.14 (VCC); no longer C27.1
- net DATA0: now also U29.2 (O0)
- net DATA1: now also U29.5 (O1)
- net DATA2: now also U29.6 (O2)
- net DATA3: now also U29.9 (O3)
- net DATA4: now also U29.12 (O4)
- net DATA5: now also U29.15 (O5)
- net DATA6: now also U29.16 (O6)
- net DATA7: now also U29.19 (O7)
- net GND: now also C28.2, J5.3 (Pin_3), Q47.3 (S), R57.2, U29.10 (GND), U30.7 (GND)
- net ~{RESET_SIGNAL}: now also U20.9 (~{MR}), U30.9 (~{MR})
- net at U20.1 (DSA): now also U20.2 (DSB), J5.1 (Pin_1)
- net at U20.10 (Q4): now also U29.8 (D3)
- net at U20.11 (Q5): now also U29.13 (D4)
- net at U20.12 (Q6): now also U29.14 (D5)
- net at U20.13 (Q7): now also U29.17 (D6), U30.1 (DSA), U30.2 (DSB)
- net at U20.4 (Q1): now also U29.3 (D0)
- net at U20.5 (Q2): now also U29.4 (D1)
- net at U20.6 (Q3): now also U29.7 (D2)
- net at U20.8 (CP): now also D2.2 (A), Q47.1 (D), R58.2, U30.8 (CP)
- net at U9.11 (4Y): now also U12.11
- net at U12.10: now also U29.1 (OE)
- net at U12.8: now also U29.11 (Cp)
- net at U12.9: now also C27.1, D2.1 (K), R57.1
- new net: J5.5 (Pin_5), Q47.2 (G)
- new net: U29.18 (D7), U30.3 (Q0)
Other:
- moved on the sheet: C18, C19, C20, C21, C26, D1, D3, D4, D5, D7, Q1, Q3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
