File: z80_schematic.kicad_sch (KiCad schematic)
At the start: 187 parts, among them J1 Port_A, J2 Port_B, J3 Conn_01x08_Socket, J4 Conn_01x03_Socket, J5 KB_conn, Q1 PMOS, Q10 PMOS, Q11 PMOS, Q12 PMOS, Q13 PMOS, Q14 NMOS, Q15 NMOS, Q16 NMOS, Q17 NMOS, Q18 PMOS, Q19 PMOS, Q2 PMOS, Q20 PMOS, Q21 PMOS, Q22 PMOS, Q23 PMOS, Q24 NMOS, Q25 NMOS, Q26 PMOS, Q27 PMOS, Q28 PMOS, Q29 PMOS, Q3 PMOS, Q30 PMOS, Q31 NMOS, Q32 PMOS, Q33 PMOS, Q34 PMOS, Q35 PMOS, Q36 NMOS, Q37 PMOS, Q38 PMOS, Q39 PMOS, Q4 PMOS, Q40 PMOS, Q41 NMOS, Q42 PMOS, Q43 PMOS, Q44 PMOS, Q45 PMOS, Q46 NMOS, Q47 NMOS, Q5 PMOS, Q6 PMOS, Q7 PMOS, Q8 PMOS, Q9 PMOS, SW1 RESET, SW2 CLK_STEP, U1 Z80CPU, U10 AT28C64B-15PU, U11 W49F002, U12 74HC14, U13 74HCT273, U14 SN74AC32, U15 SN74AC32, U16 SN74AC32, U17 SN74ACT08N, U18 SN74AC32, U19 27C512, U2 Z84C20, U20 74HC164, U21 D148K, U22 27C512, U23 D148K, U24 D148K, U25 D148K, U26 D148K, U27 27C512, U28 D148K, U29 74HCT374, U3 TC551001CP-70L, U30 74HC164, U4 EN29F040A, U5 W27E512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

Commit message: updatus
Parts:
- added SW3: SW_SP3T, symbol Switch:SW_SP3T
Connections:
- net 200Hz_CLK: now also SW3.2
- net CLK: now also SW3.3; no longer U6.3 (Q)
- net GND: now also U19.20 (~{CE}), U22.20 (~{CE}), U27.20 (~{CE})
- new net 1MHz_CLK: SW3.1
- new net CLK_SINGLE: SW3.4, U6.3 (Q)
Other:
- note added: "Clock sources Single pulses 200Hz 1MHz"
- note added: "Signal line indicators"
- note removed: "Signal lines indicators"
- moved on the sheet: C11, C2, C4, R2, R4, SW2, U6
