File: z80_schematic.kicad_sch (KiCad schematic)
At the start: 188 parts, among them J1 Port_A, J2 Port_B, J3 Conn_01x08_Socket, J4 Conn_01x03_Socket, J5 KB_conn, Q1 PMOS, Q10 PMOS, Q11 PMOS, Q12 PMOS, Q13 PMOS, Q14 NMOS, Q15 NMOS, Q16 NMOS, Q17 NMOS, Q18 PMOS, Q19 PMOS, Q2 PMOS, Q20 PMOS, Q21 PMOS, Q22 PMOS, Q23 PMOS, Q24 NMOS, Q25 NMOS, Q26 PMOS, Q27 PMOS, Q28 PMOS, Q29 PMOS, Q3 PMOS, Q30 PMOS, Q31 NMOS, Q32 PMOS, Q33 PMOS, Q34 PMOS, Q35 PMOS, Q36 NMOS, Q37 PMOS, Q38 PMOS, Q39 PMOS, Q4 PMOS, Q40 PMOS, Q41 NMOS, Q42 PMOS, Q43 PMOS, Q44 PMOS, Q45 PMOS, Q46 NMOS, Q47 NMOS, Q5 PMOS, Q6 PMOS, Q7 PMOS, Q8 PMOS, Q9 PMOS, SW1 RESET, SW2 CLK_STEP, SW3 SW_SP3T, U1 Z80CPU, U10 AT28C64B-15PU, U11 W49F002, U12 74HC14, U13 74HCT273, U14 SN74AC32, U15 SN74AC32, U16 SN74AC32, U17 SN74ACT08N, U18 SN74AC32, U19 27C512, U2 Z84C20, U20 74HC164, U21 D148K, U22 27C512, U23 D148K, U24 D148K, U25 D148K, U26 D148K, U27 27C512, U28 D148K, U29 74HCT374, U3 TC551001CP-70L, U30 74HC164, U4 EN29F040A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

Commit message: v1.1
Parts:
- removed C1, C16, C21, C23, C26, C28: 100n, symbol Device:C
- removed C27: 10n, symbol Device:C
- removed D1, D10, D11, D12, D13, D3, D4, D5, D6, D7, D8, D9: LED, symbol Device:LED
- removed D14, D15, D16, D17: LED_YELLOW, symbol Device:LED
- removed D2: D, symbol Device:D
- removed J3: Conn_01x08_Socket, Connector_PinSocket_2.54mm:PinSocket_1x08_P2.54mm_Vertical, symbol Connector:Conn_01x08_Socket
- removed J4: Conn_01x03_Socket, Connector_PinSocket_2.54mm:PinSocket_1x03_P2.54mm_Vertical, symbol Connector:Conn_01x03_Socket
- removed J5: KB_conn, symbol Connector:Conn_01x06_Socket
- removed Q1, Q10, Q11, Q12, Q3, Q4, Q5, Q6, Q7, Q8, Q9: PMOS, Package_TO_SOT_THT:TO-92, symbol Simulation_SPICE:PMOS
- removed Q14, Q15, Q16, Q17, Q47: NMOS, Package_TO_SOT_THT:TO-92, symbol Simulation_SPICE:NMOS
- removed R10, R17, R19, R20, R21, R22, R23, R24, R25, R26, R27, R28, R30, R31, R33: 1k, symbol Device:R
- removed R57: 47k, symbol Device:R
- removed R58: 10k, symbol Device:R
- removed SW3: SW_SP3T, symbol Switch:SW_SP3T
- removed U13: 74HCT273, Package_DIP:DIP-20_W7.62mm_Socket_LongPads, symbol 74xx:74HCT273
- removed U14, U16, U18: SN74AC32, Package_DIP:DIP-14_W7.62mm_Socket_LongPads, symbol Custom_symbole:SN74AC32
- removed U17: SN74ACT08N, Package_DIP:DIP-14_W7.62mm_Socket_LongPads, symbol Custom_symbole:SN74ACT08N
- removed U19, U22, U27: 27C512, Package_DIP:DIP-28_W15.24mm_Socket_LongPads, symbol Memory_EPROM:27C512
- removed U20, U30: 74HC164, Package_DIP:DIP-14_W7.62mm_Socket_LongPads, symbol 74xx:74HC164
- removed U29: 74HCT374, Package_DIP:DIP-20_W7.62mm_Socket_LongPads, symbol 74xx:74HCT374
- removed U4: EN29F040A, Package_DIP:DIP-32_W15.24mm_Socket_LongPads, symbol Custom_symbole:EN29F040A
- removed U7: 74HC374, Package_DIP:DIP-20_W7.62mm_Socket_LongPads, symbol 74xx:74HC374
- added C29: 150p, symbol Device:C
- added C30: 47p, symbol Device:C
- added C31, C32, C34, C35, C37, C38: 100n, symbol Device:C
- added C33: 1u, symbol Device:C
- added D23, D24, D25, D26, D27, D28, D29, D30, D31, D32, D33, D34, D36, D37, D38: LED, symbol Device:LED
- added J4: B_Port_A, Connector_PinHeader_2.54mm:PinHeader_1x10_P2.54mm_Vertical, symbol Connector:Conn_01x10_Socket
- added J6: B_Port_B, Connector_PinHeader_2.54mm:PinHeader_1x10_P2.54mm_Vertical, symbol Connector:Conn_01x10_Socket
- added JP1: CPU_buffer_enable, TestPoint:TestPoint_2Pads_Pitch2.54mm_Drill0.8mm, symbol Jumper:Jumper_2_Bridged
- added L1: 470u, symbol Device:L
- added Q1, Q3, Q4: NMOS, symbol Simulation_SPICE:NMOS
- added Q14, Q16, Q49, Q50, Q51, Q52, Q53, Q54, Q55, Q56, Q57: PMOS, Package_TO_SOT_THT:TO-92, symbol Simulation_SPICE:PMOS
- added Q48: Q_NPN_EBC, symbol Transistor_BJT:Q_NPN_EBC
- added R106, R108, R110, R111, R114, R115, R116, R117, R122, R123, R124, R125, R130, R131, R134, R64, R65, R66, R67, R68, R69, R70, R71, R72, R73, R74, R75, R76, R77, R78, R79, R80, R81, R82, R83, R84, R85, R86: 100, symbol Device:R
- added R107, R109, R112, R113, R118, R119, R120, R121, R126, R127, R128, R129, R132, R133, R135, R62: 1k, symbol Device:R
- added R59: 68k, symbol Device:R
- added R60, R63: 4k7, symbol Device:R
- added R61: 20k, symbol Device:R
- added SW3: SW_DPDT_x2, symbol Switch:SW_DPDT_x2
- added U13, U19, U20: ATF16V8Bxx-xxPU, Package_DIP:DIP-20_W7.62mm_Socket_LongPads, symbol Logic_Programmable:ATF16V8Bxx-xxPU
- added U14: NE555P, Package_DIP:DIP-8_W7.62mm_Socket_LongPads, symbol Timer:NE555P
- added U16, U17, U4, U7: 74LS241, Package_DIP:DIP-20_W7.62mm_Socket_LongPads, symbol 74xx:74LS241
- added U31: Z84C20, Package_DIP:DIP-40_W15.24mm_Socket_LongPads, symbol Interface:Z84C20
- J1: value Port_A -> A_Port_A
- J2: value Port_B -> A_Port_B
- R12: value 1k -> 6k8
- R29: value 1k -> 10k
- R9: value 1k -> 100
Connections:
- net RAM_PAGE_SEL_2 is gone; now on net RAM_PAGE_SEL_1: U15.1 (1A)
- net +5V: now also C14.2, R9.1, C34.1, C35.1, C37.1, C38.1, D36.2 (A), D37.2 (A), D38.2 (A), JP1.1 (A), Q14.3 (S), Q16.3 (S), Q49.3 (S), Q50.3 (S), Q51.3 (S), Q52.3 (S), Q53.3 (S), Q54.3 (S), Q55.3 (S), Q56.3 (S), Q57.3 (S), R59.1, R60.1, SW3.4 (A), U13.20 (V_{CC}), U14.4 (R), U14.8 (VCC), U16.19 (OEb), U16.20 (VCC), U17.19 (OEb), U17.20 (VCC), U19.20 (V_{CC}), U20.20 (V_{CC}), U31.26 (VCC), U4.20 (VCC), U7.20 (VCC); no longer C14.1, C18.1, C19.1, R9.2
- net 1MHz_CLK: now also U12.2, SW3.1 (A)
- net ADR0: now also U13.2 (I1), U31.6 (B/~{A}), U4.18 (O0a); no longer U1.30 (A0)
- net ADR1: now also U13.3 (I2), U31.5 (C/~{D}), U4.16 (O1a); no longer U1.31 (A1)
- net ADR10: now also U19.4 (I3), U7.14 (O2a); no longer U1.40 (A10)
- net ADR11: now also U19.5 (I4), U7.12 (O3a); no longer U1.1 (A11)
- net ADR12: now also U19.6 (I5), U7.9 (O0b); no longer U1.2 (A12)
- net ADR13: now also U19.7 (I6), U7.7 (O1b); no longer U1.3 (A13)
- net ADR14: now also U3.3 (A14), U19.8 (I7), U7.5 (O2b); no longer U1.4 (A14)
- net ADR15: now also U9.1 (1A), U19.9 (I8), U7.3 (O3b); no longer U1.5 (A15)
- net ADR2: now also U13.4 (I3), U4.14 (O2a); no longer U1.32 (A2)
- net ADR3: now also U13.5 (I4), U4.12 (O3a); no longer U1.33 (A3)
- net ADR4: now also U13.6 (I5), U4.9 (O0b); no longer U1.34 (A4)
- net ADR5: now also U13.7 (I6), U4.7 (O1b); no longer U1.35 (A5)
- net ADR6: now also U13.8 (I7), U4.5 (O2b); no longer U1.36 (A6)
- net ADR7: now also U13.9 (I8), U4.3 (O3b); no longer U1.37 (A7)
- net ADR8: now also U19.2 (I1), U7.18 (O0a); no longer U1.38 (A8)
- net ADR9: now also U19.3 (I2), U7.16 (O1a); no longer U1.39 (A9)
- net BIOS_LATCH: now also U17.6 (I2a)
- net CLK: now also SW3.2 (B), U17.8 (I3a), U31.25 (CLK)
- net CLK_SINGLE: now also SW3.3 (C)
- net DATA0: now also U20.2 (I1), U31.19 (D0)
- net DATA1: now also U20.3 (I2), U31.20 (D1)
- net DATA2: now also U20.4 (I3), U31.1 (D2)
- net DATA3: now also U20.5 (I4), U31.40 (D3)
- net DATA4: now also U20.6 (I5), U31.39 (D4)
- net DATA5: now also U20.7 (I6), U31.38 (D5)
- net DATA6: now also U20.8 (I7), U31.3 (D6)
- net DATA7: now also U20.9 (I8), U31.2 (D7)
- net GND: now also C14.1, R29.2, U15.10 (3B), U15.12 (4A), U15.13 (4B), U15.9 (3A), U5.22 (~{OE}), U9.10 (3B), U9.12 (4A), U9.13 (4B), U9.9 (3A), C29.2, C30.2, C33.1, C34.2, C35.2, C37.2, C38.2, Q1.3 (S), Q3.3 (S), Q4.3 (S), R107.1, R109.1, R112.1, R113.1, R118.1, R119.1, R120.1, R121.1, R126.1, R127.1, R128.1, R129.1, R62.2, R63.2, SW3.6 (C), U13.10 (GND), U14.1 (GND), U16.10 (GND), U17.10 (GND), U17.2 (I0a), U19.10 (GND), U20.10 (GND), U31.11 (GND), U4.1 (OEa), U4.10 (GND), U7.1 (OEa), U7.10 (GND); no longer C14.2, R12.1, R29.1
- net RAM_PAGE_SEL_0: now also U15.4 (2A), U8.15 (O5); no longer U15.9 (3A)
- net RAM_PAGE_SEL_1: now also U8.16 (O6); no longer U15.4 (2A)
- net RAM_PAGE_SEL_OVERRIDE: now also U9.3 (1Y), U17.4 (I1a); no longer U15.10 (3B)
- net ~{BIOS_CE}: now also U17.15 (I2b)
- net ~{BIOS_MAIN_CE}: now also U17.13 (I1b)
- net ~{INT}: now also U16.11 (I0b), U31.23 (~{INT})
- net ~{IORQ}: now also U16.8 (I3a), U31.36 (~{IORQ})
- net ~{M1}: now also U16.13 (I1b), U31.37 (~{M1})
- net ~{MREQ}: now also U16.6 (I2a); no longer U5.22 (~{OE})
- net ~{RAM_CE}: now also U17.17 (I3b)
- net ~{READ}: now also U16.2 (I0a), U31.35 (~{RD}); no longer U12.5
- net ~{RESET_SIGNAL}: now also U17.11 (I0b)
- net ~{WRITE}: now also U16.4 (I1a)
- net at U15.8 (3Y): no longer U3.3 (A14)
- net at U12.4: now also U9.2 (1B)
- net at Q22.2 (G): now also R83.2
- net at Q13.1 (D): now also D23.2 (A)
- net at U12.6: no longer U9.13 (4B)
- net at Q39.2 (G), Q46.2 (G): now also R86.2
- net at Q28.2 (G): now also R65.2
- net at Q21.2 (G): now also R82.2
- net at Q29.2 (G), Q36.2 (G): now also U19.19 (I/O)
- net at U12.11: no longer U9.11 (4Y)
- net at U12.12, U9.4 (2A): no longer U9.1 (1A), U9.9 (3A)
- net at R32.2: now also U31.24 (IEI)
- net at Q27.2 (G): now also R64.2
- net at Q30.2 (G): now also R66.2
- net at Q32.2 (G): now also R67.2
- net at Q33.2 (G): now also R68.2
- net at Q34.2 (G): now also R69.2
- net at Q35.2 (G): now also R70.2
- net at U12.1: now also C31.1, Q48.3 (C), R60.2
- net at Q38.2 (G): now also R72.2
- net at Q45.2 (G): now also R77.2
- net at Q23.2 (G): now also R84.2
- net at Q18.2 (G): now also R78.2
- net at Q25.2 (G), Q26.2 (G): now also R85.2
- net at U2.24 (IEI): now also U31.22 (IEO)
- net at R12.2: now also C18.1, U14.2 (TR), U14.6 (THR)
- net at Q44.2 (G): now also R76.2
- net at Q2.2 (G): now also R79.2
- net at Q37.2 (G): now also R71.2
- net at Q40.2 (G): now also R73.2
- net at Q42.2 (G): now also R74.2
- net at Q43.2 (G): now also R75.2
- net at Q19.2 (G): now also R80.2
- net at Q20.2 (G): now also R81.2
- net ARDY renamed A_ARDY
- net BRDY renamed A_BRDY
- net DISPLAY: no longer names the net of U5.19 (I/O7)
- net DISPLAY: no longer U9.10 (3B)
- net KEYBOARD renamed ~{I/O_CE_2}
- net ~{I/O_CE_2}: now also U16.17 (I3b), U31.4 (~{CE}); no longer U9.12 (4A)
- net PA0 renamed A_PA0
- net PA1 renamed A_PA1
- net PA2 renamed A_PA2
- net PA3 renamed A_PA3
- net PA4 renamed A_PA4
- net PA5 renamed A_PA5
- net PA6 renamed A_PA6
- net PA7 renamed A_PA7
- net PB0 renamed A_PB0
- net PB1 renamed A_PB1
- net PB2 renamed A_PB2
- net PB3 renamed A_PB3
- net PB4 renamed A_PB4
- net PB5 renamed A_PB5
- net PB6 renamed A_PB6
- net PB7 renamed A_PB7
- net RAM/FLASH_LATCH: no longer names the net of U5.17 (I/O5)
- net RAM/FLASH_LATCH: no longer U9.2 (1B)
- net ~{ASTB} renamed ~{A_ASTB}
- net ~{BSTB} renamed ~{A_BSTB}
- net ~{FLASH_CE}: no longer names the net of Q13.2 (G)
- net ~{FLASH_CE}: now also R106.2; no longer U5.15 (I/O3)
- net ~{I/O_CE} renamed ~{I/O_CE_1}
- net ~{I/O_CE_1}: now also U5.15 (I/O3), U16.15 (I2b)
- new net: D25.1 (K), R112.2
- new net: D25.2 (A), Q16.1 (D)
- new net: R66.1, U19.14 (I/O)
- new net: R134.1, U17.16 (O1a)
- new net: Q4.2 (G), R134.2
- new net: D23.1 (K), R107.2
- new net: R78.1, U13.12 (I/O)
- new net: D32.1 (K), R127.2
- new net: Q3.1 (D), R133.1
- new net: Q3.2 (G), R131.2
- new net: R117.1, U16.3 (O3b)
- new net: Q53.2 (G), R117.2
- new net: D27.2 (A), Q50.1 (D)
- new net: Q50.2 (G), R114.2
- new net: R64.1, U19.12 (I/O)
- new net: D34.1 (K), R129.2
- new net: D36.1 (K), R132.2
- new net: C32.1, Q48.2 (B), R59.2, R61.1
- new net: R76.1, U20.17 (I/O)
- new net: R130.1, U17.12 (O3a)
- new net: R131.1, U17.14 (O2a)
- new net: R125.1, U17.3 (O3b)
- new net: R124.1, U17.5 (O2b)
- new net: R123.1, U17.7 (O1b)
- new net: R122.1, U17.9 (O0b)
- new net: R110.1, U16.14 (O2a)
- new net: Q16.2 (G), R110.2
- new net: D28.2 (A), Q51.1 (D)
- new net: Q51.2 (G), R115.2
- new net: D32.2 (A), Q55.1 (D)
- new net: Q55.2 (G), R123.2
- new net: D27.1 (K), R118.2
- new net: D31.1 (K), R126.2
- new net: D33.2 (A), Q56.1 (D)
- new net: Q56.2 (G), R124.2
- new net: R71.1, U20.12 (I/O)
- new net: R72.1, U20.13 (I/O)
- new net: R73.1, U20.14 (I/O)
- new net: R74.1, U20.15 (I/O)
- new net: R75.1, U20.16 (I/O)
- new net: R77.1, U20.18 (I/O)
- new net: R86.1, U20.19 (I/O)
- new net: R82.1, U13.16 (I/O)
- new net: R69.1, U19.17 (I/O)
- new net: D31.2 (A), Q54.1 (D)
- new net: D26.1 (K), R113.2
- new net: Q1.1 (D), R132.1
- new net: D24.2 (A), Q14.1 (D)
- new net: Q14.2 (G), R108.2
- new net: D30.1 (K), R121.2
- new net: D29.1 (K), R120.2
- new net: Q1.2 (G), R130.2
- new net: R84.1, U13.18 (I/O)
- new net: Q54.2 (G), R122.2
- new net: D34.2 (A), Q57.1 (D)
- new net: Q57.2 (G), R125.2
- new net: D38.1 (K), R135.2
- new net: U1.2 (A12), U7.11 (I0b)
- new net: U1.3 (A13), U7.13 (I1b)
- new net: U1.4 (A14), U7.15 (I2b)
- new net: U1.5 (A15), U7.17 (I3b)
- new net: JP1.2 (B), R29.1, U4.19 (OEb), U7.19 (OEb)
- new net: U1.38 (A8), U7.2 (I0a)
- new net: U1.39 (A9), U7.4 (I1a)
- new net: U1.40 (A10), U7.6 (I2a)
- new net: U1.1 (A11), U7.8 (I3a)
- new net: C29.1, C31.2, L1.1
- new net: C30.1, C32.2, L1.2
- new net: R65.1, U19.13 (I/O)
- new net: R67.1, U19.15 (I/O)
- new net: R68.1, U19.16 (I/O)
- new net: R70.1, U19.18 (I/O)
- new net: D28.1 (K), R119.2
- new net: D37.1 (K), R133.2
- new net: Q4.1 (D), R135.1
- new net: R80.1, U13.14 (I/O)
- new net: R111.1, U16.12 (O3a)
- new net: Q49.2 (G), R111.2
- new net: R79.1, U13.13 (I/O)
- new net: R81.1, U13.15 (I/O)
- new net: R83.1, U13.17 (I/O)
- new net: R85.1, U13.19 (I/O)
- new net: U1.34 (A4), U4.11 (I0b)
- new net: U1.35 (A5), U4.13 (I1b)
- new net: U1.36 (A6), U4.15 (I2b)
- new net: U1.37 (A7), U4.17 (I3b)
- new net: U1.30 (A0), U4.2 (I0a)
- new net: U1.31 (A1), U4.4 (I1a)
- new net: U1.32 (A2), U4.6 (I2a)
- new net: U1.33 (A3), U4.8 (I3a)
- new net: C19.1, U14.5 (CV)
- new net: R12.1, R9.2, U14.7 (DIS)
- new net: D30.2 (A), Q53.1 (D)
- new net: D24.1 (K), R109.2
- new net: R116.1, U16.5 (O2b)
- new net: Q52.2 (G), R116.2
- new net: R115.1, U16.7 (O1b)
- new net: D33.1 (K), R128.2
- new net: R108.1, U16.16 (O1a)
- new net: R61.2, R63.1
- new net: C33.2, Q48.1 (E), R62.1
- new net: D29.2 (A), Q52.1 (D)
- new net: R114.1, U16.9 (O0b)
- new net: R106.1, U16.18 (O0a)
- new net: D26.2 (A), Q49.1 (D)
- new net 1kHz_CLK: U13.1 (I), U14.3 (Q), U19.1 (I), U20.1 (I)
- new net B_ARDY: J4.9 (Pin_9), U31.18 (ARDY)
- new net B_BRDY: J6.9 (Pin_9), U31.21 (BRDY)
- new net B_PA0: J4.1 (Pin_1), U31.15 (PA0)
- new net B_PA1: J4.2 (Pin_2), U31.14 (PA1)
- new net B_PA2: J4.3 (Pin_3), U31.13 (PA2)
- new net B_PA3: J4.4 (Pin_4), U31.12 (PA3)
- new net B_PA4: J4.5 (Pin_5), U31.10 (PA4)
- new net B_PA5: J4.6 (Pin_6), U31.9 (PA5)
- new net B_PA6: J4.7 (Pin_7), U31.8 (PA6)
- new net B_PA7: J4.8 (Pin_8), U31.7 (PA7)
- new net B_PB0: J6.1 (Pin_1), U31.27 (PB0)
- new net B_PB1: J6.2 (Pin_2), U31.28 (PB1)
- new net B_PB2: J6.3 (Pin_3), U31.29 (PB2)
- new net B_PB3: J6.4 (Pin_4), U31.30 (PB3)
- new net B_PB4: J6.5 (Pin_5), U31.31 (PB4)
- new net B_PB5: J6.6 (Pin_6), U31.32 (PB5)
- new net B_PB6: J6.7 (Pin_7), U31.33 (PB6)
- new net B_PB7: J6.8 (Pin_8), U31.34 (PB7)
- new net MONITOR_EN: SW3.5 (B), U13.11 (I9), U16.1 (OEa), U17.1 (OEa), U19.11 (I9), U20.11 (I9)
- new net ~{B_ASTB}: J4.10 (Pin_10), U31.16 (~{ASTB})
- new net ~{B_BSTB}: J6.10 (Pin_10), U31.17 (~{BSTB})
- no-connect marks 4 -> 11
Other:
- note added: "ADDRESS SPACE (64kB, divided into 4 main 16kB segments) 0000 - 3FFF EEPROM BIOS 0000 - 1FFF BIOS MAIN 2000 - 3FFF BIOS PAGED (32 pages, 256kB total memory) 4000 - BFFF RAM (4 pages, 128kB total memory) C000 - FFFF Misc (I/O, page switching) + LAST 8kB OF RAM (ALWAYS AVAILABLE) I/O chip 1: C000 Port A, Data C001 Port B, Data C002 Port A, Command C003 Port B, Command I/O chip 2: C004 Port A, Data C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"
- note added: "Clock sources Single pulses 1MHz"
- note added: "I/O chip 1"
- note added: "I/O chip 2"
- note added: "TC551001CP - 128kB RAM W49F002 - 256kB PAGED BIOS AT28C64 - 16kB MAIN BIOS W27E512 - 64kB CHIP SELECT"
- note removed: "ADDRESS SPACE (64kB, divided into 4 main 16kB segments) 0000 - 3FFF EEPROM BIOS 0000 - 1FFF BIOS MAIN 2000 - 3FFF BIOS PAGED (32 pages, 256kB total memory) 4000 - 7FFF RAM (8 pages, 128kB total memory) 8000 - BFFF FLASH program memory (32 pages, 512kB total memory) C000 - FFFF Misc (I/O, page switching) + LAST 8kB OF RAM (ALWAYS AVAILABLE) I/O chip: C000 Port A, Data C001 Port B, Data C002 Port A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"
- note removed: "Clock sources Single pulses 200Hz 1MHz"
- note removed: "EN29F040 - 512kB FLASH TC551001CP - 128kB RAM W49F002 - 256kB PAGED BIOS AT28C64 - 16kB MAIN BIOS W27E512 - 64kB CHIP SELECT"
- note removed: "FLASH"
- note removed: "I/O chip"
- note removed: "I/O_CE address decoding"
- note removed: "LCD display output"
- note removed: "PS/2 keyboard input with interrupt"
- note removed: "RAM/FLASH"
- moved on the sheet: C10, C17, C22, C24, C25, C8, C9, J1, J2, Q27, Q28, Q29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

Commit message: v1.2
Parts:
- removed C14, C18, C19, C22, C24: 100n, symbol Device:C
- removed J1: A_Port_A, Connector_PinHeader_2.54mm:PinHeader_1x10_P2.54mm_Vertical, symbol Connector:Conn_01x10_Socket
- removed J2: A_Port_B, Connector_PinHeader_2.54mm:PinHeader_1x10_P2.54mm_Vertical, symbol Connector:Conn_01x10_Socket
- removed J4: B_Port_A, Connector_PinHeader_2.54mm:PinHeader_1x10_P2.54mm_Vertical, symbol Connector:Conn_01x10_Socket
- removed J6: B_Port_B, Connector_PinHeader_2.54mm:PinHeader_1x10_P2.54mm_Vertical, symbol Connector:Conn_01x10_Socket
- removed JP1: CPU_buffer_enable, TestPoint:TestPoint_2Pads_Pitch2.54mm_Drill0.8mm, symbol Jumper:Jumper_2_Bridged
- removed Q18, Q19, Q2, Q20, Q21, Q22, Q23, Q26, Q27, Q28, Q29, Q30, Q32, Q33, Q34, Q35, Q37, Q38, Q39, Q40, Q42, Q43, Q44: PMOS, Package_TO_SOT_THT:TO-92, symbol Simulation_SPICE:PMOS
- removed Q24, Q25, Q31, Q36, Q46: NMOS, Package_TO_SOT_THT:TO-92, symbol Simulation_SPICE:NMOS
- removed R106, R108, R110, R111, R114, R115, R116, R117, R122, R123, R124, R125, R130, R131, R134, R71, R72, R73, R74, R75, R76, R77, R78, R79, R80, R81, R82, R83, R84, R85, R86, R9: 100, symbol Device:R
- removed R12: 6k8, symbol Device:R
- removed R18, R34, R35, R36, R37, R38, R39, R41, R42, R43, R44, R45, R46, R48, R7, R8: 1k, symbol Device:R
- removed R29, R40, R47: 10k, symbol Device:R
- removed SW3: SW_DPDT_x2, symbol Switch:SW_DPDT_x2
- removed U13, U19: ATF16V8Bxx-xxPU, Package_DIP:DIP-20_W7.62mm_Socket_LongPads, symbol Logic_Programmable:ATF16V8Bxx-xxPU
- removed U14: NE555P, Package_DIP:DIP-8_W7.62mm_Socket_LongPads, symbol Timer:NE555P
- removed U21, U23, U28: D148K, Display_7Segment:D1X8K, symbol Display_Character:D148K
- added C1: 1000u, Capacitor_THT:C_Rect_L41.5mm_W11.0mm_P37.50mm_MKS4, symbol Device:C_Polarized
- added C14: 470u, Capacitor_THT:C_Radial_D10.0mm_H20.0mm_P5.00mm, symbol Device:C_Polarized
- added C16: 47u, Capacitor_THT:C_Radial_D5.0mm_H11.0mm_P2.00mm, symbol Device:C_Polarized
- added C18, C19, C21, C23, C24: 220u, Capacitor_THT:C_Radial_D6.3mm_H11.0mm_P2.50mm, symbol Device:C_Polarized
- added C26, C27, C28, C36, C39: 100n, Capacitor_THT:C_Disc_D6.0mm_W2.5mm_P5.00mm, symbol Device:C
- added C40: 1u, Capacitor_THT:C_Disc_D5.1mm_W3.2mm_P5.00mm, symbol Device:C
- added J1, J2, J4, J6: Conn_01x14_Socket, Connector_PinSocket_2.54mm:PinSocket_1x14_P2.54mm_Vertical, symbol Connector:Conn_01x14_Socket
- added J5: EXTERNAL_CLOCK, Connector_PinSocket_2.54mm:PinSocket_1x02_P2.54mm_Vertical, symbol Connector:Conn_01x02_Socket
- added J7: 5V_IN, Connector_Phoenix_MSTB:PhoenixContact_MSTBVA_2,5_2-G_1x02_P5.00mm_Vertical, symbol Connector:Conn_01x02_Socket
- added Q42, Q43, Q44, Q90, Q98: 2N7002, Package_TO_SOT_SMD:SOT-23, symbol Transistor_FET:2N7002
- added Q46, Q47, Q58, Q59, Q60, Q61, Q62, Q63, Q64, Q65, Q66, Q67, Q68, Q69, Q70, Q71, Q72, Q73, Q74, Q75, Q76, Q77, Q78, Q79, Q80, Q81, Q82, Q83, Q84, Q85, Q86, Q87, Q88, Q89, Q91, Q92, Q93, Q94, Q95, Q96, Q97: BSS84, Package_TO_SOT_SMD:SOT-23, symbol Transistor_FET:BSS84
- added R136, R137, R138, R139, R140, R141, R142, R151, R152, R153, R154, R155, R156, R157, R166, R167, R168, R169, R170, R171, R172, R57, R58, R94, R95, R96, R97: 1k, Resistor_SMD:R_1206_3216Metric_Pad1.30x1.75mm_HandSolder, symbol Device:R
- added SW3: SW_SPST, Connector_Phoenix_MSTB:PhoenixContact_MSTBVA_2,5_2-G_1x02_P5.00mm_Vertical, symbol Switch:SW_SPST
- added SW4: ADDR_BUS_BUFFERS, Library:SPDT_SWITCH_OS102011MS2QN1, symbol Switch:SW_SPDT
- added SW5: SW_SPDT, Library:SPDT_SWITCH_OS102011MS2QN1, symbol Switch:SW_SPDT
- added SW6: CLOCK_SEL, Library:SPDT_SWITCH_OS102011MS2QN1, symbol Switch:SW_SPDT
- added SW8: CLK_SOURCE_SEL, Library:SPDT_SWITCH_OS102011MS2QN1, symbol Switch:SW_SPDT
- added U21, U22, U23, U28, U30: ATF16V8Bxx-xxPU, Package_DIP:DIP-20_W7.62mm_Socket_LongPads, symbol Logic_Programmable:ATF16V8Bxx-xxPU
- added U27, U29, U32: D148K, Display_7Segment:D1X8K, symbol Display_Character:D148K
- C10, C11, C12, C13, C15, C17, C2, C20, C25, C3, C30, C31, C32, C34, C35, C37, C38, C5, C6, C7, C8, C9: footprint (none) -> Capacitor_THT:C_Disc_D6.0mm_W2.5mm_P5.00mm
- C29, C4: footprint (none) -> Capacitor_THT:C_Disc_D3.8mm_W2.6mm_P2.50mm
- C33: footprint (none) -> Capacitor_THT:C_Disc_D5.1mm_W3.2mm_P5.00mm
- D23, D24, D25, D26, D27, D28, D29, D30, D31, D32, D33, D34, D36, D37, D38: footprint (none) -> LED_THT:LED_D5.0mm
- L1: footprint (none) -> Inductor_THT:L_Axial_L11.0mm_D4.5mm_P15.24mm_Horizontal_Fastron_MECC
- Q1, Q3, Q4: value NMOS -> 2N7002; footprint (none) -> Package_TO_SOT_SMD:SOT-23; symbol Simulation_SPICE:NMOS -> Transistor_FET:2N7002
- Q13, Q14, Q16, Q45, Q49, Q50, Q51, Q52, Q53, Q54, Q55, Q56, Q57: value PMOS -> BSS84; footprint Package_TO_SOT_THT:TO-92 -> Package_TO_SOT_SMD:SOT-23; symbol Simulation_SPICE:PMOS -> Transistor_FET:BSS84
- Q41: value NMOS -> 2N7002; footprint Package_TO_SOT_THT:TO-92 -> Package_TO_SOT_SMD:SOT-23; symbol Simulation_SPICE:NMOS -> Transistor_FET:2N7002
- Q48: footprint (none) -> Package_TO_SOT_THT:TO-18-3
- R1, R107, R109, R11, R112, R113, R118, R119, R120, R121, R126, R127, R128, R129, R13, R132, R133, R135, R14, R15, R32, R4, R49, R5, R50, R51, R52, R53, R54, R56, R6, R62: footprint (none) -> Resistor_SMD:R_1206_3216Metric_Pad1.30x1.75mm_HandSolder
- R16, R3, R59, R60, R61, R63: footprint (none) -> Resistor_THT:R_Axial_DIN0411_L9.9mm_D3.6mm_P15.24mm_Horizontal
- R2: footprint (none) -> Resistor_THT:R_Axial_DIN0204_L3.6mm_D1.6mm_P7.62mm_Horizontal
- R55: value 10k -> 1k; footprint (none) -> Resistor_SMD:R_1206_3216Metric_Pad1.30x1.75mm_HandSolder
- R64, R65, R66, R67, R68, R69, R70: value 100 -> 1k; footprint (none) -> Resistor_SMD:R_1206_3216Metric_Pad1.30x1.75mm_HandSolder
- SW1, SW2: footprint (none) -> Button_Switch_THT:SW_PUSH_6mm_H5mm
- U1: footprint Package_DIP:DIP-40_W15.24mm_Socket_LongPads -> Socket:DIP_Socket-40_W11.9mm_W12.7mm_W15.24mm_W17.78mm_W18.5mm_3M_240-1280-00-0602J
- U10: footprint 28P6_ATM -> Socket:DIP_Socket-28_W11.9mm_W12.7mm_W15.24mm_W17.78mm_W18.5mm_3M_228-1277-00-0602J; KiLib_Generator (none) -> connector/DIP_socket
- U11: footprint Package_DIP:DIP-32_W15.24mm_Socket_LongPads -> Socket:DIP_Socket-32_W11.9mm_W12.7mm_W15.24mm_W17.78mm_W18.5mm_3M_232-1285-00-0602J
- U3: footprint Package_DIP:DIP-32_W15.24mm_Socket_LongPads -> Socket:DIP_Socket-32_W11.9mm_W12.7mm_W15.24mm_W17.78mm_W18.5mm_3M_232-1285-00-0602J; KiLib_Generator (none) -> connector/DIP_socket
- U5: footprint Package_DIP:DIP-28_W15.24mm_Socket_LongPads -> Socket:DIP_Socket-28_W11.9mm_W12.7mm_W15.24mm_W17.78mm_W18.5mm_3M_228-1277-00-0602J; KiLib_Generator (none) -> connector/DIP_socket
Connections:
- net 1kHz_CLK is gone; now on net +5V: U20.1 (I)
- net +5V: now also Q13.2 (S), Q14.2 (S), Q16.2 (S), Q45.2 (S), Q49.2 (S), Q50.2 (S), Q51.2 (S), Q52.2 (S), Q53.2 (S), Q54.2 (S), Q55.2 (S), Q56.2 (S), Q57.2 (S), U20.6 (I5), U20.7 (I6), U20.8 (I7), U20.9 (I8), C1.1, C14.1, C16.1, C18.1, C19.1, C21.1, C23.1, C24.1, C26.1, C27.1, C28.1, C36.1, C39.1, C40.2, J1.1 (Pin_1), J1.2 (Pin_2), J2.1 (Pin_1), J2.2 (Pin_2), J4.1 (Pin_1), J4.2 (Pin_2), J6.1 (Pin_1), J6.2 (Pin_2), Q46.2 (S), Q47.2 (S), Q58.2 (S), Q59.2 (S), Q60.2 (S), Q61.2 (S), Q62.2 (S), Q63.2 (S), Q64.2 (S), Q65.2 (S), Q66.2 (S), Q67.2 (S), Q68.2 (S), Q69.2 (S), Q70.2 (S), Q71.2 (S), Q72.2 (S), Q73.2 (S), Q74.2 (S), Q75.2 (S), Q76.2 (S), Q77.2 (S), Q78.2 (S), Q79.2 (S), Q80.2 (S), Q81.2 (S), Q82.2 (S), Q83.2 (S), Q84.2 (S), Q85.2 (S), Q86.2 (S), Q87.2 (S), Q88.2 (S), Q89.2 (S), Q91.2 (S), Q92.2 (S), Q93.2 (S), Q94.2 (S), Q95.2 (S), Q96.2 (S), Q97.2 (S), SW3.2 (B), SW4.1 (A), SW5.1 (A), U21.1 (I), U21.20 (V_{CC}), U21.6 (I5), U21.7 (I6), U21.8 (I7), U21.9 (I8), U22.1 (I), U22.20 (V_{CC}), U22.6 (I5), U22.7 (I6), U22.8 (I7), U22.9 (I8), U23.1 (I), U23.20 (V_{CC}), U23.6 (I5), U23.7 (I6), U23.8 (I7), U23.9 (I8), U28.1 (I), U28.20 (V_{CC}), U28.6 (I5), U28.7 (I6), U28.8 (I7), U28.9 (I8), U30.1 (I), U30.20 (V_{CC}), U30.6 (I5), U30.7 (I6), U30.8 (I7), U30.9 (I8); no longer Q13.3 (S), Q14.3 (S), Q16.3 (S), Q45.3 (S), Q49.3 (S), Q50.3 (S), Q51.3 (S), Q52.3 (S), Q53.3 (S), Q54.3 (S), Q55.3 (S), Q56.3 (S), Q57.3 (S), U16.19 (OEb), U17.19 (OEb)
- net 1MHz_CLK: now also U12.6, SW8.3 (C); no longer U12.2
- net ADR0: now also U21.2 (I1)
- net ADR1: now also U21.3 (I2)
- net ADR10: now also U23.4 (I3)
- net ADR11: now also U23.5 (I4)
- net ADR12: now also U20.2 (I1)
- net ADR13: now also U20.3 (I2)
- net ADR14: now also U20.4 (I3)
- net ADR15: now also U20.5 (I4)
- net ADR2: now also U21.4 (I3)
- net ADR3: now also U21.5 (I4)
- net ADR4: now also U22.2 (I1)
- net ADR5: now also U22.3 (I2)
- net ADR6: now also U22.4 (I3)
- net ADR7: now also U22.5 (I4)
- net ADR8: now also U23.2 (I1)
- net ADR9: now also U23.3 (I2)
- net A_ARDY: now also J1.13 (Pin_13)
- net A_BRDY: now also J2.13 (Pin_13)
- net A_PA0: now also J1.5 (Pin_5)
- net A_PA1: now also J1.6 (Pin_6)
- net A_PA2: now also J1.7 (Pin_7)
- net A_PA3: now also J1.8 (Pin_8)
- net A_PA4: now also J1.9 (Pin_9)
- net A_PA5: now also J1.10 (Pin_10)
- net A_PA6: now also J1.11 (Pin_11)
- net A_PA7: now also J1.12 (Pin_12)
- net A_PB0: now also J2.5 (Pin_5)
- net A_PB1: now also J2.6 (Pin_6)
- net A_PB2: now also J2.7 (Pin_7)
- net A_PB3: now also J2.8 (Pin_8)
- net A_PB4: now also J2.9 (Pin_9)
- net A_PB5: now also J2.10 (Pin_10)
- net A_PB6: now also J2.11 (Pin_11)
- net A_PB7: now also J2.12 (Pin_12)
- net B_ARDY: now also J4.13 (Pin_13)
- net B_BRDY: now also J6.13 (Pin_13)
- net B_PA0: now also J4.5 (Pin_5)
- net B_PA1: now also J4.6 (Pin_6)
- net B_PA2: now also J4.7 (Pin_7)
- net B_PA3: now also J4.8 (Pin_8)
- net B_PA4: now also J4.9 (Pin_9)
- net B_PA5: now also J4.10 (Pin_10)
- net B_PA6: now also J4.11 (Pin_11)
- net B_PA7: now also J4.12 (Pin_12)
- net B_PB0: now also J6.5 (Pin_5)
- net B_PB1: now also J6.6 (Pin_6)
- net B_PB2: now also J6.7 (Pin_7)
- net B_PB3: now also J6.8 (Pin_8)
- net B_PB4: now also J6.9 (Pin_9)
- net B_PB5: now also J6.10 (Pin_10)
- net B_PB6: now also J6.11 (Pin_11)
- net B_PB7: now also J6.12 (Pin_12)
- net CLK: now also SW6.2 (B)
- net CLK_SINGLE: now also SW6.3 (C)
- net DATA0: now also U28.2 (I1); no longer U20.2 (I1)
- net DATA1: now also U28.3 (I2); no longer U20.3 (I2)
- net DATA2: now also U28.4 (I3); no longer U20.4 (I3)
- net DATA3: now also U28.5 (I4); no longer U20.5 (I4)
- net DATA4: now also U30.2 (I1); no longer U20.6 (I5)
- net DATA5: now also U30.3 (I2); no longer U20.7 (I6)
- net DATA6: now also U30.4 (I3); no longer U20.8 (I7)
- net DATA7: now also U30.5 (I4); no longer U20.9 (I8)
- net GND: now also Q1.2 (S), Q3.2 (S), Q4.2 (S), Q41.2 (S), U12.11, C1.2, C14.2, C16.2, C18.2, C19.2, C21.2, C23.2, C24.2, C26.2, C27.2, C28.2, C36.2, C39.2, C40.1, J1.3 (Pin_3), J1.4 (Pin_4), J2.3 (Pin_3), J2.4 (Pin_4), J4.3 (Pin_3), J4.4 (Pin_4), J5.1 (Pin_1), J6.3 (Pin_3), J6.4 (Pin_4), J7.1 (Pin_1), Q42.2 (S), Q43.2 (S), Q44.2 (S), Q90.2 (S), Q98.2 (S), SW4.3 (C), SW5.3 (C), U21.10 (GND), U22.10 (GND), U23.10 (GND), U28.10 (GND), U30.10 (GND); no longer Q1.3 (S), Q3.3 (S), Q4.3 (S), Q41.3 (S), R55.1, U4.1 (OEa), U7.1 (OEa)
- net MONITOR_EN: now also U12.2, U16.19 (OEb), U17.19 (OEb), U21.11 (I9), U22.11 (I9), U23.11 (I9), U28.11 (I9), U30.11 (I9); no longer U16.1 (OEa), U17.1 (OEa)
- net ~{A_ASTB}: now also J1.14 (Pin_14)
- net ~{A_BSTB}: now also J2.14 (Pin_14)
- net ~{B_ASTB}: now also J4.14 (Pin_14)
- net ~{B_BSTB}: now also J6.14 (Pin_14)
- net at D25.2 (A): now also Q16.3 (D); no longer Q16.1 (D)
- net at R66.1: now also Q67.3 (D)
- net at R66.2: now also U25.9 (F)
- net at U17.16 (O1a): now also Q4.1 (G)
- net at R6.2, U1.17 (~{NMI}): now also U1.24 (~{WAIT}), U1.25 (~{BUSRQ})
- net at U26.1 (E): now also R95.2; no longer U25.1 (E)
- net at U26.10 (G): now also R97.2; no longer U25.10 (G)
- net at U26.2 (D): now also R94.2; no longer U25.2 (D)
- net at U25.3 (CC), U25.8 (CC): now also Q42.3 (D)
- net at U26.4 (C): now also R70.2; no longer U25.4 (C)
- net at U26.6 (B): now also R69.2; no longer U25.6 (B)
- net at U26.7 (A): now also R68.2; no longer U25.7 (A)
- net at U26.9 (F): now also R96.2; no longer U25.9 (F)
- net at Q3.1 (G): now also U17.14 (O2a); no longer R133.1
- net at U12.5: now also C31.1, Q48.3 (C), R60.2
- net at U16.3 (O3b): now also Q53.1 (G)
- net at R65.2: now also U25.1 (E)
- net at Q50.1 (G): now also U16.9 (O0b); no longer D27.2 (A)
- net at R64.1: now also Q65.3 (D)
- net at R64.2: now also U25.2 (D)
- net at U20.17 (I/O): now also Q60.1 (G)
- net at U17.12 (O3a): now also Q1.1 (G)
- net at U17.3 (O3b): now also Q57.1 (G)
- net at U17.5 (O2b): now also Q56.1 (G)
- net at U17.7 (O1b): now also Q55.1 (G)
- net at U17.9 (O0b): now also Q54.1 (G)
- net at U16.14 (O2a): now also Q16.1 (G)
- net at Q51.1 (G): now also U16.7 (O1b); no longer D28.2 (A)
- net at D23.2 (A): now also Q13.3 (D); no longer Q13.1 (D)
- net at D32.2 (A): now also Q55.3 (D); no longer Q55.1 (D)
- net at D33.2 (A): now also Q56.3 (D); no longer Q56.1 (D)
- net at U20.12 (I/O): now also Q45.1 (G)
- net at U20.13 (I/O): now also Q46.1 (G)
- net at U20.14 (I/O): now also Q47.1 (G)
- net at U20.15 (I/O): now also Q58.1 (G)
- net at U20.16 (I/O): now also Q59.1 (G)
- net at U20.18 (I/O): now also Q61.1 (G)
- net at U20.19 (I/O): now also Q41.1 (G)
- net at U24.3 (CC), U24.8 (CC): now also Q41.3 (D); no longer Q41.1 (D)
- net at R69.1: now also Q70.3 (D)
- net at R50.1: now also Q46.3 (D)
- net at D31.2 (A): now also Q54.3 (D); no longer Q54.1 (D)
- net at R132.1: now also Q1.3 (D); no longer Q1.1 (D)
- net at Q14.1 (G): now also U16.16 (O1a); no longer D24.2 (A)
- net at R56.1: now also Q61.3 (D); no longer Q45.1 (D)
- net at R55.2: now also U25.7 (A); no longer Q41.2 (G)
- net at D34.2 (A): now also Q57.3 (D); no longer Q57.1 (D)
- net at R54.1: now also Q60.3 (D)
- net at U4.19 (OEb), U7.19 (OEb): now also U12.9, SW4.2 (B)
- net at U7.2 (I0a): now also U1.1 (A11); no longer U1.38 (A8)
- net at U7.4 (I1a): now also U1.38 (A8); no longer U1.39 (A9)
- net at U7.6 (I2a): now also U1.39 (A9); no longer U1.40 (A10)
- net at U7.8 (I3a): now also U1.40 (A10); no longer U1.1 (A11)
- net at R65.1: now also Q66.3 (D)
- net at R67.1: now also Q68.3 (D)
- net at R68.1: now also Q69.3 (D)
- net at R70.1: now also Q71.3 (D)
- net at U12.8: now also U4.1 (OEa), U7.1 (OEa)
- net at R67.2: now also U25.10 (G)
- net at U26.3 (CC), U26.8 (CC): now also Q43.3 (D)
- net at R135.1: now also Q4.3 (D); no longer Q4.1 (D)
- net at R49.1: now also Q45.3 (D)
- net at U16.12 (O3a): now also Q49.1 (G)
- net at U4.11 (I0b): now also U1.37 (A7); no longer U1.34 (A4)
- net at U4.13 (I1b): now also U1.36 (A6); no longer U1.35 (A5)
- net at U4.15 (I2b): now also U1.34 (A4); no longer U1.36 (A6)
- net at U4.17 (I3b): now also U1.32 (A2); no longer U1.37 (A7)
- net at U4.6 (I2a): now also U1.33 (A3); no longer U1.32 (A2)
- net at U4.8 (I3a): now also U1.35 (A5); no longer U1.33 (A3)
- net at D30.2 (A): now also Q53.3 (D); no longer Q53.1 (D)
- net at R52.1: now also Q58.3 (D)
- net at R53.1: now also Q59.3 (D)
- net at U16.5 (O2b): now also Q52.1 (G)
- net at R51.1: now also Q47.3 (D)
- net at D29.2 (A): now also Q52.3 (D); no longer Q52.1 (D)
- net at U16.18 (O0a): now also Q13.1 (G)
- net at D26.2 (A): now also Q49.3 (D); no longer Q49.1 (D)
- new net: Q88.3 (D), R156.1
- new net: R156.2, U29.9 (F)
- new net: Q43.1 (G), U22.19 (I/O)
- new net: Q85.3 (D), R153.1
- new net: R153.2, U29.4 (C)
- new net: SW6.1 (A), SW8.2 (B)
- new net: Q3.3 (D), R133.1
- new net: Q81.3 (D), R141.1
- new net: R141.2, U27.9 (F)
- new net: Q68.1 (G), U21.18 (I/O)
- new net: D27.2 (A), Q50.3 (D)
- new net: Q76.1 (G), U23.12 (I/O)
- new net: Q77.1 (G), U23.13 (I/O)
- new net: Q78.1 (G), U23.14 (I/O)
- new net: Q79.1 (G), U23.15 (I/O)
- new net: Q80.1 (G), U23.16 (I/O)
- new net: Q81.1 (G), U23.17 (I/O)
- new net: Q82.1 (G), U23.18 (I/O)
- new net: Q44.1 (G), U23.19 (I/O)
- new net: J7.2 (Pin_2), SW3.1 (A)
- new net: Q80.3 (D), R140.1
- new net: R140.2, U27.1 (E)
- new net: Q69.1 (G), U22.12 (I/O)
- new net: D28.2 (A), Q51.3 (D)
- new net: Q74.3 (D), R96.1
- new net: Q96.1 (G), U30.17 (I/O)
- new net: Q96.3 (D), R171.1
- new net: Q73.3 (D), R95.1
- new net: Q89.3 (D), R157.1
- new net: R157.2, U29.10 (G)
- new net: Q85.1 (G), U28.14 (I/O)
- new net: Q75.3 (D), R97.1
- new net: Q95.3 (D), R170.1
- new net: R170.2, U32.1 (E)
- new net: Q91.1 (G), U30.12 (I/O)
- new net: Q91.3 (D), R166.1
- new net: R155.2, U29.1 (E)
- new net: R154.2, U29.2 (D)
- new net: Q90.3 (D), U29.3 (CC), U29.8 (CC)
- new net: R152.2, U29.6 (B)
- new net: R151.2, U29.7 (A)
- new net: Q77.3 (D), R137.1
- new net: D24.2 (A), Q14.3 (D)
- new net: Q97.3 (D), R172.1
- new net: R172.2, U32.10 (G)
- new net: Q74.1 (G), U22.17 (I/O)
- new net: Q64.1 (G), U21.14 (I/O)
- new net: Q64.3 (D), R58.1
- new net: Q78.3 (D), R138.1
- new net: Q73.1 (G), U22.16 (I/O)
- new net: Q82.3 (D), R142.1
- new net: Q75.1 (G), U22.18 (I/O)
- new net: Q44.3 (D), U27.3 (CC), U27.8 (CC)
- new net: Q76.3 (D), R136.1
- new net: R136.2, U27.7 (A)
- new net: R142.2, U27.10 (G)
- new net: R139.2, U27.2 (D)
- new net: R138.2, U27.4 (C)
- new net: R137.2, U27.6 (B)
- new net: Q42.1 (G), U21.19 (I/O)
- new net: Q83.3 (D), R151.1
- new net: Q72.1 (G), U22.15 (I/O)
- new net: Q72.3 (D), R94.1
- new net: Q89.1 (G), U28.18 (I/O)
- new net: R166.2, U32.7 (A)
- new net: Q63.3 (D), R57.1
- new net: R57.2, U25.6 (B)
- new net: Q62.1 (G), U21.12 (I/O)
- new net: Q62.3 (D), R55.1
- new net: J5.2 (Pin_2), SW8.1 (A)
- new net: Q97.1 (G), U30.18 (I/O)
- new net: Q93.3 (D), R168.1
- new net: R168.2, U32.4 (C)
- new net: Q65.1 (G), U21.15 (I/O)
- new net: R58.2, U25.4 (C)
- new net: Q79.3 (D), R139.1
- new net: R169.2, U32.2 (D)
- new net: Q98.3 (D), U32.3 (CC), U32.8 (CC)
- new net: R167.2, U32.6 (B)
- new net: R171.2, U32.9 (F)
- new net: Q87.1 (G), U28.16 (I/O)
- new net: Q87.3 (D), R155.1
- new net: Q84.3 (D), R152.1
- new net: Q86.1 (G), U28.15 (I/O)
- new net: Q86.3 (D), R154.1
- new net: Q84.1 (G), U28.13 (I/O)
- new net: Q66.1 (G), U21.16 (I/O)
- new net: Q92.3 (D), R167.1
- new net: Q63.1 (G), U21.13 (I/O)
- new net: Q67.1 (G), U21.17 (I/O)
- new net: Q98.1 (G), U30.19 (I/O)
- new net: Q71.1 (G), U22.14 (I/O)
- new net: Q95.1 (G), U30.16 (I/O)
- new net: Q70.1 (G), U22.13 (I/O)
- new net: Q83.1 (G), U28.12 (I/O)
- new net: Q88.1 (G), U28.17 (I/O)
- new net: Q90.1 (G), U28.19 (I/O)
- new net: Q92.1 (G), U30.13 (I/O)
- new net: Q93.1 (G), U30.14 (I/O)
- new net: Q94.1 (G), U30.15 (I/O)
- new net: Q94.3 (D), R169.1
- new net ~{MONITOR_EN}: SW5.2 (B), U12.1, U16.1 (OEa), U17.1 (OEa)
Other:
- note added: "ADDRESS 0 - 3 hex decoding"
- note added: "ADDRESS 12 - 15 hex decoding"
- note added: "ADDRESS 4 - 7 hex decoding"
- note added: "ADDRESS 8 - 11 hex decoding"
- note added: "Clock sources Single pulses 1MHz / EXTERNAL"
- note added: "DATA 0 - 3 hex decoding"
- note added: "DATA 3 - 7 hex decoding"
- note removed: "ADDR 0 - 7 hex decoding"
- note removed: "ADDR 8 - 15 hex decoding"
- note removed: "Clock sources Single pulses 1MHz"
- note removed: "DATA 0 - 7 hex decoding"
- moved on the sheet: C25, Q41, Q45, R49, R50, R51, R52, R53, R54, R56, R6, U12D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

Commit message: changes
Connections:
- net GND: no longer U15.10 (3B), U15.12 (4A), U15.13 (4B), U15.9 (3A)
- net ~{MREQ}: now also U15.10 (3B), U15.12 (4A)
- net ~{READ}: now also U15.9 (3A); no longer U10.22 (~{OE}), U11.24 (~{OE}), U3.24 (~{OE})
- net ~{WRITE}: now also U15.13 (4B); no longer U12.13, U3.29 (R/~{W})
- net ~{MWRITE}: now reaches U15.11 (4Y)
- net ~{MWRITE}: now also U12.13, U3.29 (R/~{W})
- net ~{MREAD}: now reaches U15.8 (3Y)
- net ~{MREAD}: now also U10.22 (~{OE}), U11.24 (~{OE}), U3.24 (~{OE})
