File: z80_schematic.kicad_pcb (KiCad board)
At the start: 4 copper layers, 206.2 x 170.2 mm, 234 parts, among them J1 Conn_01x14_Socket, J2 Conn_01x14_Socket, J4 Conn_01x14_Socket, J5 EXTERNAL_CLOCK, J6 Conn_01x14_Socket, J7 5V_IN, Q1 2N7002, Q13 BSS84, Q14 BSS84, Q16 BSS84, Q3 2N7002, Q4 2N7002, Q41 2N7002, Q42 2N7002, Q43 2N7002, Q44 2N7002, Q45 BSS84, Q46 BSS84, Q47 BSS84, Q48 Q_NPN_EBC, Q49 BSS84, Q50 BSS84, Q51 BSS84, Q52 BSS84, Q53 BSS84, Q54 BSS84, Q55 BSS84, Q56 BSS84, Q57 BSS84, Q58 BSS84, Q59 BSS84, Q60 BSS84, Q61 BSS84, Q62 BSS84, Q63 BSS84, Q64 BSS84, Q65 BSS84, Q66 BSS84, Q67 BSS84, Q68 BSS84, Q69 BSS84, Q70 BSS84, Q71 BSS84, Q72 BSS84, Q73 BSS84, Q74 BSS84, Q75 BSS84, Q76 BSS84, Q77 BSS84, Q78 BSS84, Q79 BSS84, Q80 BSS84, Q81 BSS84, Q82 BSS84, Q83 BSS84, Q84 BSS84, Q85 BSS84, Q86 BSS84, Q87 BSS84, Q88 BSS84, Q89 BSS84, Q90 2N7002, Q91 BSS84, Q92 BSS84, Q93 BSS84, Q94 BSS84, Q95 BSS84, Q96 BSS84, Q97 BSS84, Q98 2N7002, SW1 RESET, SW2 CLK_STEP, SW3 SW_SPST, SW4 ADDR_BUS_BUFFERS, SW5 SW_SPDT, SW6 CLOCK_SEL, SW8 CLK_SOURCE_SEL, U1 Z80CPU, U10 AT28C64B-15PU, U11 W49F002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

Commit message: changes
Connections:
- U10 pad 22: ~{READ} -> ~{MREAD}
- U11 pad 24: ~{READ} -> ~{MREAD}
- U12 pad 13: ~{WRITE} -> ~{MWRITE}
- U15 pad 10: GND -> ~{MREQ}
- U15 pad 11: unconnected-(U15-4Y-Pad11) -> ~{MWRITE}
- U15 pad 12: GND -> ~{MREQ}
- U15 pad 13: GND -> ~{WRITE}
- U15 pad 8: unconnected-(U15-3Y-Pad8) -> ~{MREAD}
- U15 pad 9: GND -> ~{READ}
- U3 pad 24: ~{READ} -> ~{MREAD}
- U3 pad 29: ~{WRITE} -> ~{MWRITE}
Routing:
- net ~{MWRITE}: track 0.00 -> 189.3 mm, vias 0 -> 6
- net ~{MREAD}: track 0.00 -> 130.5 mm, vias 0 -> 7
- net ~{MREQ}: track 28.4 -> 146.4 mm, vias 1 -> 5
- net ~{WRITE}: track 204.8 -> 158.4 mm, vias 9 -> 2
- net ~{READ}: track 260.7 -> 271.5 mm, vias 11 -> 8
Other:
- board text added: "+ -"
- board text added: "PWR SW"
- board text added: "Z80 COMPUTER by Dominik Dworak Address space: 0000 - 3FFF Main BIOS 2000 - 3FFF Paged BIOS | 4000 - BFFF Paged RAM | C000 - C003 PIO 1 C004 - C007 PIO 2 | C008 - Paging Latch | E000 - FFFF Last 8kB of RAM (1E000 - 1FFFF)"
- board text added: "^ ADDRESS BUS ^"
- board text added: "^ DATA BUS ^"
